File: jhl_synth0.kicad_pcb (KiCad board)
At the start: 2 copper layers, 4 parts, among them U1 YAAJ_BluePill, U2 YAAJ_BlackPill

Commit message: 作図中
Parts:
- added J1: Conn_01x04, Connector_PinSocket_2.54mm:PinSocket_1x04_P2.54mm_Vertical, F.Cu at (377.8, 104.5)
- added J3: Conn_01x04, Connector_PinSocket_2.54mm:PinSocket_1x04_P2.54mm_Vertical, F.Cu at (382.4, 104.5)
- added J4: Conn_01x04, Connector_PinSocket_2.54mm:PinSocket_1x04_P2.54mm_Vertical, F.Cu at (387.0, 104.5)
- added J7: Conn_01x07, Connector_PinSocket_2.54mm:PinSocket_1x07_P2.54mm_Vertical, F.Cu at (373.2, 104.5)
- added JP1: SolderJumper_2_Bridged, Jumper:SolderJumper-2_P1.3mm_Bridged_RoundedPad1.0x1.5mm, F.Cu at (377.6, 116.2)
- added JP2: SolderJumper_2_Bridged, Jumper:SolderJumper-2_P1.3mm_Bridged_RoundedPad1.0x1.5mm, F.Cu at (377.6, 119.8)
- added RV1: R_Potentiometer, Potentiometer_THT:Potentiometer_Vishay_T73YP_Vertical, F.Cu at (325.1, 108.8)
- added RV10: R_Potentiometer, Potentiometer_THT:Potentiometer_Vishay_T93YA_Vertical, F.Cu at (340.9, 132.8)
- added RV11: R_Potentiometer, Potentiometer_THT:Potentiometer_Vishay_T73YP_Vertical, F.Cu at (333.6, 108.8)
- added RV12: R_Potentiometer, Potentiometer_THT:Potentiometer_Vishay_T93YA_Vertical, F.Cu at (340.9, 139.6)
- added RV13: R_Potentiometer, Potentiometer_THT:Potentiometer_Vishay_T73YP_Vertical, F.Cu at (333.6, 117.0)
- added RV14: R_Potentiometer, Potentiometer_THT:Potentiometer_Vishay_T93YA_Vertical, F.Cu at (352.2, 105.7)
- added RV15: R_Potentiometer, Potentiometer_THT:Potentiometer_Vishay_T73YP_Vertical, F.Cu at (333.6, 125.1)
- added RV16: R_Potentiometer, Potentiometer_THT:Potentiometer_Vishay_T93YA_Vertical, F.Cu at (352.2, 112.5)
- added RV17: R_Potentiometer, Potentiometer_THT:Potentiometer_Vishay_T73YP_Vertical, F.Cu at (333.6, 133.3)
- added RV18: R_Potentiometer, Potentiometer_THT:Potentiometer_Vishay_T73YP_Vertical, F.Cu at (333.6, 141.4)
- added RV19: R_Potentiometer, Potentiometer_THT:Potentiometer_Vishay_T93YA_Vertical, F.Cu at (352.2, 119.3)
- added RV2: R_Potentiometer, Potentiometer_THT:Potentiometer_Vishay_T93YA_Vertical, F.Cu at (340.9, 105.7)
- added RV20: R_Potentiometer, Potentiometer_THT:Potentiometer_Vishay_T93YA_Vertical, F.Cu at (352.2, 126.0)
- added RV3: R_Potentiometer, Potentiometer_THT:Potentiometer_Vishay_T73YP_Vertical, F.Cu at (325.1, 117.0)
- added RV4: R_Potentiometer, Potentiometer_THT:Potentiometer_Vishay_T93YA_Vertical, F.Cu at (340.9, 112.5)
- added RV5: R_Potentiometer, Potentiometer_THT:Potentiometer_Vishay_T73YP_Vertical, F.Cu at (325.1, 125.1)
- added RV6: R_Potentiometer, Potentiometer_THT:Potentiometer_Vishay_T93YA_Vertical, F.Cu at (340.9, 119.3)
- added RV7: R_Potentiometer, Potentiometer_THT:Potentiometer_Vishay_T73YP_Vertical, F.Cu at (325.1, 133.3)
- added RV8: R_Potentiometer, Potentiometer_THT:Potentiometer_Vishay_T93YA_Vertical, F.Cu at (340.9, 126.0)
- added RV9: R_Potentiometer, Potentiometer_THT:Potentiometer_Vishay_T73YP_Vertical, F.Cu at (325.1, 141.4)
- added SW1: SW_SPST, Button_Switch_SMD:SW_Push_1P1T_XKB_TS-1187A, F.Cu at (364.6, 105.5)
- added SW10: SW_SPST, Button_Switch_THT:SW_TH_Tactile_Omron_B3F-110x, F.Cu at (312.0, 142.8)
- added SW11: SW_SPST, Button_Switch_SMD:SW_Push_1P1T_XKB_TS-1187A, F.Cu at (364.6, 138.8)
- added SW12: SW_SPST, Button_Switch_THT:SW_TH_Tactile_Omron_B3F-110x, F.Cu at (312.0, 152.4)
- added SW2: SW_SPST, Button_Switch_THT:SW_TH_Tactile_Omron_B3F-110x, F.Cu at (312.0, 104.0)
- added SW3: SW_SPST, Button_Switch_SMD:SW_Push_1P1T_XKB_TS-1187A, F.Cu at (364.6, 112.2)
- added SW4: SW_SPST, Button_Switch_THT:SW_TH_Tactile_Omron_B3F-110x, F.Cu at (312.0, 113.7)
- added SW5: SW_SPST, Button_Switch_SMD:SW_Push_1P1T_XKB_TS-1187A, F.Cu at (364.6, 118.8)
- added SW6: SW_SPST, Button_Switch_THT:SW_TH_Tactile_Omron_B3F-110x, F.Cu at (312.0, 123.3)
- added SW7: SW_SPST, Button_Switch_SMD:SW_Push_1P1T_XKB_TS-1187A, F.Cu at (364.6, 125.5)
- added SW8: SW_SPST, Button_Switch_THT:SW_TH_Tactile_Omron_B3F-110x, F.Cu at (312.0, 133.1)
- added SW9: SW_SPST, Button_Switch_SMD:SW_Push_1P1T_XKB_TS-1187A, F.Cu at (364.6, 132.2)
Connections:
- A1 pad 10: unconnected-(A1-A1-Pad10) -> a1
- A1 pad 11: unconnected-(A1-A2-Pad11) -> a2
- A1 pad 12: unconnected-(A1-A3-Pad12) -> a3
- A1 pad 13: unconnected-(A1-A4-Pad13) -> a4
- A1 pad 14: unconnected-(A1-A5-Pad14) -> SPI_SCLK
- A1 pad 17: unconnected-(A1-D2/SDA-Pad17) -> I2C_SDA
- A1 pad 18: unconnected-(A1-D3/SCL-Pad18) -> I2C_SCL
- A1 pad 19: unconnected-(A1-D4-Pad19) -> sw0
- A1 pad 20: unconnected-(A1-D5-Pad20) -> sw1
- A1 pad 21: unconnected-(A1-D6-Pad21) -> sw2
- A1 pad 22: unconnected-(A1-D7-Pad22) -> sw3
- A1 pad 23: unconnected-(A1-D8-Pad23) -> sw4
- A1 pad 24: unconnected-(A1-D9-Pad24) -> sw5
- A1 pad 29: unconnected-(A1-GND-Pad29) -> GND
- A1 pad 30: unconnected-(A1-AREF-Pad30) -> avref
- A1 pad 4: unconnected-(A1-3V3-Pad4) -> +3.3V
- A1 pad 5: unconnected-(A1-+5V-Pad5) -> +5VP
- A1 pad 6: unconnected-(A1-GND-Pad6) -> GND
- A1 pad 7: unconnected-(A1-GND-Pad7) -> GND
- A1 pad 9: unconnected-(A1-A0-Pad9) -> a0
- A2 pad 10: unconnected-(A2-D7-Pad10) -> sw3
- A2 pad 11: unconnected-(A2-D8-Pad11) -> sw4
- A2 pad 12: unconnected-(A2-D9-Pad12) -> sw5
- A2 pad 17: unconnected-(A2-3V3-Pad17) -> +3.3V
- A2 pad 18: unconnected-(A2-AREF-Pad18) -> avref
- A2 pad 19: unconnected-(A2-A0-Pad19) -> a0
- A2 pad 20: unconnected-(A2-A1-Pad20) -> a1
- A2 pad 21: unconnected-(A2-A2-Pad21) -> a2
- A2 pad 22: unconnected-(A2-A3-Pad22) -> a3
- A2 pad 23: unconnected-(A2-A4-Pad23) -> a4
- A2 pad 24: unconnected-(A2-A5-Pad24) -> SPI_SCLK
- A2 pad 25: unconnected-(A2-A6-Pad25) -> SPI_MOSI
- A2 pad 26: unconnected-(A2-A7-Pad26) -> SPI_MISO
- A2 pad 27: unconnected-(A2-+5V-Pad27) -> +5VP
- A2 pad 29: unconnected-(A2-GND-Pad29) -> GND
- A2 pad 4: unconnected-(A2-GND-Pad4) -> GND
- A2 pad 5: unconnected-(A2-D2-Pad5) -> I2C_SDA
- A2 pad 6: unconnected-(A2-D3-Pad6) -> I2C_SCL
- A2 pad 7: unconnected-(A2-D4-Pad7) -> sw0
- A2 pad 8: unconnected-(A2-D5-Pad8) -> sw1
- A2 pad 9: unconnected-(A2-D6-Pad9) -> sw2
- U1 pad 10: unconnected-(U1-PA15-Pad10) -> SPI_SS
- U1 pad 14: unconnected-(U1-PB6-Pad14) -> I2C_SCL
- U1 pad 15: unconnected-(U1-PB7-Pad15) -> I2C_SDA
- U1 pad 18: unconnected-(U1-5V-Pad18) -> +5VP
- U1 pad 19: unconnected-(U1-GND-Pad19) -> GND
- U1 pad 20: unconnected-(U1-3V3-Pad20) -> +3.3V
- U1 pad 25: unconnected-(U1-PA0-Pad25) -> a0
- U1 pad 26: unconnected-(U1-PA1-Pad26) -> a1
- U1 pad 27: unconnected-(U1-PA2-Pad27) -> a2
- U1 pad 28: unconnected-(U1-PA3-Pad28) -> a3
- U1 pad 29: unconnected-(U1-PA4-Pad29) -> a4
- U1 pad 30: unconnected-(U1-PA5-Pad30) -> SPI_SCLK
- U1 pad 31: unconnected-(U1-PA6-Pad31) -> SPI_MOSI
- U1 pad 32: unconnected-(U1-PA7-Pad32) -> SPI_MISO
- U1 pad 33: unconnected-(U1-PB0-Pad33) -> a8
- U1 pad 34: unconnected-(U1-PB1-Pad34) -> a9
- U1 pad 38: unconnected-(U1-3V3-Pad38) -> +3.3V
- U1 pad 39: unconnected-(U1-GND-Pad39) -> GND
- U1 pad 40: unconnected-(U1-GND-Pad40) -> GND
- U2 pad 10: unconnected-(U2-PA15-Pad10) -> SPI_SS
- U2 pad 14: unconnected-(U2-PB6-Pad14) -> I2C_SCL
- U2 pad 15: unconnected-(U2-PB7-Pad15) -> I2C_SDA
- U2 pad 16: unconnected-(U2-3V3-Pad16) -> +3.3V
- U2 pad 17: unconnected-(U2-GND-Pad17) -> GND
- U2 pad 18: unconnected-(U2-GND-Pad18) -> GND
- U2 pad 23: unconnected-(U2-PA0-Pad23) -> a0
- U2 pad 24: unconnected-(U2-PA1-Pad24) -> a1
- U2 pad 25: unconnected-(U2-PA2-Pad25) -> a2
- U2 pad 26: unconnected-(U2-PA3-Pad26) -> a3
- U2 pad 27: unconnected-(U2-PA4-Pad27) -> a4
- U2 pad 28: unconnected-(U2-PA5-Pad28) -> SPI_SCLK
- U2 pad 29: unconnected-(U2-PA6-Pad29) -> SPI_MOSI
- U2 pad 30: unconnected-(U2-PA7-Pad30) -> SPI_MISO
- U2 pad 31: unconnected-(U2-PB0-Pad31) -> a8
- U2 pad 32: unconnected-(U2-PB1-Pad32) -> a9

Commit message: 仮回路、仮配置
Parts:
- added J2: USB_B_Micro, Connector_USB:USB_Micro-B_Molex-105017-0001, F.Cu at (173.5, 50.0)
- added J5: Conn_01x01, Connector_PinSocket_2.54mm:PinSocket_1x01_P2.54mm_Vertical, F.Cu at (167.0, 49.5)
- added JP3: SolderJumper_2_Bridged, Jumper:SolderJumper-2_P1.3mm_Bridged_RoundedPad1.0x1.5mm, F.Cu at (172.0, 56.0)
- added JP4: SolderJumper_2_Bridged, Jumper:SolderJumper-2_P1.3mm_Bridged_RoundedPad1.0x1.5mm, F.Cu at (173.0, 58.5)
- moved JP1 268.2 mm to (113.0, 73.0)
- moved SW11 253.6 mm to (115.5, 91.2), turned to -90 degrees
- moved SW9 242.6 mm to (125.5, 91.0), turned to -90 degrees
- moved SW7 233.3 mm to (133.8, 91.0), turned to -90 degrees
- moved RV2 226.3 mm to (116.0, 79.9), turned to 180 degrees
- moved JP2 225.8 mm to (160.5, 58.0)
- moved SW5 221.3 mm to (145.0, 91.2), turned to -90 degrees
- moved RV4 216.4 mm to (127.0, 79.8), turned to 180 degrees
- moved J4 212.3 mm to (181.2, 52.5), turned to 90 degrees
- moved SW3 211.2 mm to (154.5, 91.0), turned to -90 degrees
- moved RV1 211.1 mm to (116.0, 79.8), turned to 90 degrees
- moved RV6 206.7 mm to (138.0, 79.9), turned to 180 degrees
- moved SW12 204.9 mm to (117.5, 87.8), turned to -90 degrees
- moved RV3 201.6 mm to (126.9, 79.7), turned to 90 degrees
- moved J7 200.2 mm to (181.0, 48.5), turned to 90 degrees
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Connections:
- A1 pad 14: SPI_SCLK -> a5
- A2 pad 24: SPI_SCLK -> a5
- A2 pad 25: SPI_MOSI -> a6
- A2 pad 26: SPI_MISO -> a7
- RV1 pad 1: VDDA -> avref
- RV1 pad 3: GNDA -> GND
- RV10 pad 1: VDDA -> avref
- RV10 pad 3: GNDA -> GND
- RV11 pad 1: VDDA -> avref
- RV11 pad 2: SPI_SCLK -> a5
- RV11 pad 3: GNDA -> GND
- RV12 pad 1: VDDA -> avref
- RV12 pad 2: SPI_SCLK -> a5
- RV12 pad 3: GNDA -> GND
- RV13 pad 1: VDDA -> avref
- RV13 pad 2: SPI_MOSI -> a6
- RV13 pad 3: GNDA -> GND
- RV14 pad 1: VDDA -> avref
- RV14 pad 2: SPI_MOSI -> a6
- RV14 pad 3: GNDA -> GND
- RV15 pad 1: VDDA -> avref
- RV15 pad 2: SPI_MISO -> a7
- RV15 pad 3: GNDA -> GND
- RV16 pad 1: VDDA -> avref
- RV16 pad 2: SPI_MISO -> a7
- RV16 pad 3: GNDA -> GND
- RV17 pad 1: VDDA -> avref
- RV17 pad 3: GNDA -> GND
- RV18 pad 1: VDDA -> avref
- RV18 pad 3: GNDA -> GND
- RV19 pad 1: VDDA -> avref
- RV19 pad 3: GNDA -> GND
- RV2 pad 1: VDDA -> avref
- RV2 pad 3: GNDA -> GND
- RV20 pad 1: VDDA -> avref
- RV20 pad 3: GNDA -> GND
- RV3 pad 1: VDDA -> avref
- RV3 pad 3: GNDA -> GND
- RV4 pad 1: VDDA -> avref
- RV4 pad 3: GNDA -> GND
- RV5 pad 1: VDDA -> avref
- RV5 pad 3: GNDA -> GND
- RV6 pad 1: VDDA -> avref
- RV6 pad 3: GNDA -> GND
- RV7 pad 1: VDDA -> avref
- RV7 pad 3: GNDA -> GND
- RV8 pad 1: VDDA -> avref
- RV8 pad 3: GNDA -> GND
- RV9 pad 1: VDDA -> avref
- RV9 pad 3: GNDA -> GND
- U1 pad 11: unconnected-(U1-PB3-Pad11) -> SPI_SCLK
- U1 pad 12: unconnected-(U1-PB4-Pad12) -> SPI_MISO
- U1 pad 13: unconnected-(U1-PB5-Pad13) -> SPI_MOSI
- U1 pad 2: unconnected-(U1-PB13-Pad2) -> sw3
- U1 pad 3: unconnected-(U1-PB14-Pad3) -> sw4
- U1 pad 30: SPI_SCLK -> a5
- U1 pad 31: SPI_MOSI -> a6
- U1 pad 32: SPI_MISO -> a7
- U1 pad 4: unconnected-(U1-PB15-Pad4) -> sw5
- U1 pad 8: unconnected-(U1-PA11-Pad8) -> USB_DM
- U1 pad 9: unconnected-(U1-PA12-Pad9) -> USB_DP
- U2 pad 11: unconnected-(U2-PB3-Pad11) -> SPI_SCLK
- U2 pad 12: unconnected-(U2-PB4-Pad12) -> SPI_MISO
- U2 pad 13: unconnected-(U2-PB5-Pad13) -> SPI_MOSI
- U2 pad 2: unconnected-(U2-PB13-Pad2) -> sw3
- U2 pad 28: SPI_SCLK -> a5
- U2 pad 29: SPI_MOSI -> a6
- U2 pad 3: unconnected-(U2-PB14-Pad3) -> sw4
- U2 pad 30: SPI_MISO -> a7
- U2 pad 4: unconnected-(U2-PB15-Pad4) -> sw5
- U2 pad 8: unconnected-(U2-PA11-Pad8) -> USB_DM
- U2 pad 9: unconnected-(U2-PA12-Pad9) -> USB_DP
Routing:
- net I2C_SCL: track 0.00 -> 139.7 mm
- net I2C_SDA: track 0.00 -> 138.0 mm
- net sw5: track 0.00 -> 117.4 mm
- net sw4: track 0.00 -> 96.7 mm
- net SPI_MISO: track 0.00 -> 81.8 mm
- net SPI_MOSI: track 0.00 -> 78.3 mm
- net SPI_SS: track 0.00 -> 73.3 mm, vias 0 -> 1
- net sw3: track 0.00 -> 72.9 mm
- net sw0: track 0.00 -> 72.8 mm
- net SPI_SCLK: track 0.00 -> 68.9 mm
- net sw1: track 0.00 -> 60.5 mm
- net avref: track 0.00 -> 57.1 mm, vias 0 -> 1
- net a9: track 0.00 -> 57.0 mm
- net sw2: track 0.00 -> 55.6 mm
- net a0: track 0.00 -> 52.0 mm
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- added copper zone on In1.Cu, net GND
Other:
- copper layers 2 -> 4

Commit message: 日々の進捗
Parts:
- added C1: 0.1u, Capacitor_SMD:C_0603_1608Metric_Pad1.08x0.95mm_HandSolder, F.Cu at (261.6, 54.6)
- added D1: LED_Small_Filled, LED_SMD:LED_0603_1608Metric_Pad1.05x0.95mm_HandSolder, F.Cu at (257.3, 54.6)
- added D2: LED_Small_Filled, LED_SMD:LED_0603_1608Metric_Pad1.05x0.95mm_HandSolder, F.Cu at (257.3, 57.2)
- added D3: LED_Small_Filled, LED_SMD:LED_0603_1608Metric_Pad1.05x0.95mm_HandSolder, F.Cu at (257.3, 59.8)
- added D4: LED_Small_Filled, LED_SMD:LED_0603_1608Metric_Pad1.05x0.95mm_HandSolder, F.Cu at (257.3, 62.4)
- added IC1: HT16K33, libs:HT16K33, F.Cu at (227.3, 58.4)
- added JP5: SolderJumper_3_Bridged12, Jumper:SolderJumper-3_P1.3mm_Bridged12_RoundedPad1.0x1.5mm, F.Cu at (184.2, 54.6)
- added JP6: SolderJumper_3_Bridged12, Jumper:SolderJumper-3_P1.3mm_Bridged12_RoundedPad1.0x1.5mm, F.Cu at (177.8, 48.3)
- J7: value Conn_01x07 -> Conn_01x08; footprint Connector_PinSocket_2.54mm:PinSocket_1x07_P2.54mm_Vertical -> Connector_PinHeader_2.54mm:PinHeader_1x08_P2.54mm_Vertical
- moved RV18 37.4 mm to (238.8, 91.4)
- moved RV20 37.4 mm to (238.8, 91.4)
- moved SW1 32.5 mm to (165.1, 124.5)
- moved SW10 32.5 mm to (127.4, 120.2)
- moved SW11 32.5 mm to (115.7, 123.7)
- moved SW12 32.5 mm to (117.7, 120.2)
- moved SW2 32.5 mm to (167.2, 120.2)
- moved SW3 32.5 mm to (154.7, 123.5)
- moved SW4 32.5 mm to (156.5, 120.2)
- moved SW5 32.5 mm to (145.2, 123.7)
- moved SW6 32.5 mm to (146.8, 120.2)
- moved SW7 32.5 mm to (134.0, 123.5)
- moved SW8 32.5 mm to (137.1, 120.2)
- moved SW9 32.5 mm to (125.7, 123.5)
- moved RV17 26.7 mm to (219.7, 90.1)
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Connections:
- J3 pad 1: GND -> Net-(J3-Pin_1)
- J3 pad 2: +3.3V -> Net-(J3-Pin_2)
Routing:
- net I2C_SCL: track 139.7 -> 39.5 mm
- net avref: track 57.1 -> 154.7 mm
- net I2C_SDA: track 138.0 -> 50.8 mm
- net SPI_SS: track 73.3 -> 50.2 mm
- net sw0: track 72.8 -> 52.7 mm
- net +3.3V: track 35.1 -> 18.7 mm
- net a4: track 52.0 -> 65.2 mm
- net SPI_MISO: track 81.8 -> 72.2 mm
- net unconnected-(J2-Shield-Pad6): track 0.00 -> 9.34 mm, vias 0 -> 1
- net Net-(J2-ID): track 9.34 -> 0.00 mm, vias 1 -> 0
- net a8: track 51.3 -> 43.3 mm
- net a7: track 42.1 -> 47.0 mm
- net SPI_MOSI: track 78.3 -> 75.4 mm
- net SPI_SCLK: track 68.9 -> 67.3 mm

Commit message: 251023
Parts:
- removed the J4 at (166.3, 64.8)
- removed JP1, JP2, JP3, JP4: SolderJumper_2_Bridged, Jumper:SolderJumper-2_P1.3mm_Bridged_RoundedPad1.0x1.5mm
- removed JP5, JP6: SolderJumper_3_Bridged12, Jumper:SolderJumper-3_P1.3mm_Bridged12_RoundedPad1.0x1.5mm
- added A2: Arduino_Leonardo, Module:Arduino_UNO_R3, F.Cu at (118.1, 52.1)
- added D11: LED_Small_Filled, LED_SMD:LED_0603_1608Metric_Pad1.05x0.95mm_HandSolder, F.Cu at (132.1, 80.0)
- added D12: LED_Small_Filled, LED_SMD:LED_0603_1608Metric_Pad1.05x0.95mm_HandSolder, F.Cu at (134.6, 80.0)
- added D13: LED_Small_Filled, LED_SMD:LED_0603_1608Metric_Pad1.05x0.95mm_HandSolder, F.Cu at (138.4, 80.0)
- added D14: LED_Small_Filled, LED_SMD:LED_0603_1608Metric_Pad1.05x0.95mm_HandSolder, F.Cu at (141.0, 80.0)
- added D15: LED_Small_Filled, LED_SMD:LED_0603_1608Metric_Pad1.05x0.95mm_HandSolder, F.Cu at (143.5, 80.0)
- added D16: LED_Small_Filled, LED_SMD:LED_0603_1608Metric_Pad1.05x0.95mm_HandSolder, F.Cu at (146.1, 80.0)
- added D17: LED_Small_Filled, LED_SMD:LED_0603_1608Metric_Pad1.05x0.95mm_HandSolder, F.Cu at (149.9, 80.0)
- added D18: LED_Small_Filled, LED_SMD:LED_0603_1608Metric_Pad1.05x0.95mm_HandSolder, F.Cu at (152.4, 80.0)
- added D19: LED_Small_Filled, LED_SMD:LED_0603_1608Metric_Pad1.05x0.95mm_HandSolder, F.Cu at (154.9, 80.0)
- added D20: LED_Small_Filled, LED_SMD:LED_0603_1608Metric_Pad1.05x0.95mm_HandSolder, F.Cu at (157.5, 80.0)
- added D21: LED_Small_Filled, LED_SMD:LED_0603_1608Metric_Pad1.05x0.95mm_HandSolder, F.Cu at (161.3, 80.0)
- added D22: LED_Small_Filled, LED_SMD:LED_0603_1608Metric_Pad1.05x0.95mm_HandSolder, F.Cu at (163.8, 80.0)
- added D23: LED_Small_Filled, LED_SMD:LED_0603_1608Metric_Pad1.05x0.95mm_HandSolder, F.Cu at (166.4, 80.0)
- added D24: LED_Small_Filled, LED_SMD:LED_0603_1608Metric_Pad1.05x0.95mm_HandSolder, F.Cu at (168.9, 80.0)
- added D25: LED_Small_Filled, LED_SMD:LED_0603_1608Metric_Pad1.05x0.95mm_HandSolder, F.Cu at (104.1, 106.7)
- added D26: LED_Small_Filled, LED_SMD:LED_0603_1608Metric_Pad1.05x0.95mm_HandSolder, F.Cu at (106.7, 106.7)
- added D27: LED_Small_Filled, LED_SMD:LED_0603_1608Metric_Pad1.05x0.95mm_HandSolder, F.Cu at (109.2, 106.7)
- added D28: LED_Small_Filled, LED_SMD:LED_0603_1608Metric_Pad1.05x0.95mm_HandSolder, F.Cu at (111.8, 106.7)
- added D29: LED_Small_Filled, LED_SMD:LED_0603_1608Metric_Pad1.05x0.95mm_HandSolder, F.Cu at (115.6, 106.7)
- added D3: LED_Small_Filled, LED_SMD:LED_0603_1608Metric_Pad1.05x0.95mm_HandSolder, F.Cu at (109.2, 80.0)
- added D30: LED_Small_Filled, LED_SMD:LED_0603_1608Metric_Pad1.05x0.95mm_HandSolder, F.Cu at (118.1, 106.7)
- added D31: LED_Small_Filled, LED_SMD:LED_0603_1608Metric_Pad1.05x0.95mm_HandSolder, F.Cu at (120.7, 106.7)
- added D32: LED_Small_Filled, LED_SMD:LED_0603_1608Metric_Pad1.05x0.95mm_HandSolder, F.Cu at (123.2, 106.7)
- added D33: LED_Small_Filled, LED_SMD:LED_0603_1608Metric_Pad1.05x0.95mm_HandSolder, F.Cu at (127.0, 106.7)
- added D34: LED_Small_Filled, LED_SMD:LED_0603_1608Metric_Pad1.05x0.95mm_HandSolder, F.Cu at (129.5, 106.7)
- added D35: LED_Small_Filled, LED_SMD:LED_0603_1608Metric_Pad1.05x0.95mm_HandSolder, F.Cu at (132.1, 106.7)
- added D36: LED_Small_Filled, LED_SMD:LED_0603_1608Metric_Pad1.05x0.95mm_HandSolder, F.Cu at (134.6, 106.7)
- added D37: LED_Small_Filled, LED_SMD:LED_0603_1608Metric_Pad1.05x0.95mm_HandSolder, F.Cu at (138.4, 106.7)
- added D38: LED_Small_Filled, LED_SMD:LED_0603_1608Metric_Pad1.05x0.95mm_HandSolder, F.Cu at (141.0, 106.7)
- added D39: LED_Small_Filled, LED_SMD:LED_0603_1608Metric_Pad1.05x0.95mm_HandSolder, F.Cu at (143.5, 106.7)
- added D4: LED_Small_Filled, LED_SMD:LED_0603_1608Metric_Pad1.05x0.95mm_HandSolder, F.Cu at (111.8, 80.0)
- added D40: LED_Small_Filled, LED_SMD:LED_0603_1608Metric_Pad1.05x0.95mm_HandSolder, F.Cu at (146.1, 106.7)
- added D41: LED_Small_Filled, LED_SMD:LED_0603_1608Metric_Pad1.05x0.95mm_HandSolder, F.Cu at (243.8, 85.1)
- added D42: LED_Small_Filled, LED_SMD:LED_0603_1608Metric_Pad1.05x0.95mm_HandSolder, F.Cu at (246.4, 85.1)
- added D43: LED_Small_Filled, LED_SMD:LED_0603_1608Metric_Pad1.05x0.95mm_HandSolder, F.Cu at (250.1, 85.1)
- added D44: LED_Small_Filled, LED_SMD:LED_0603_1608Metric_Pad1.05x0.95mm_HandSolder, F.Cu at (252.7, 85.1)
- added D45: LED_Small_Filled, LED_SMD:LED_0603_1608Metric_Pad1.05x0.95mm_HandSolder, F.Cu at (255.3, 85.1)
- added D46: LED_Small_Filled, LED_SMD:LED_0603_1608Metric_Pad1.05x0.95mm_HandSolder, F.Cu at (257.9, 85.1)
- added D47: LED_Small_Filled, LED_SMD:LED_0603_1608Metric_Pad1.05x0.95mm_HandSolder, F.Cu at (224.2, 79.5)
- added D48: LED_Small_Filled, LED_SMD:LED_0603_1608Metric_Pad1.05x0.95mm_HandSolder, F.Cu at (226.8, 79.5)
- added D49: LED_Small_Filled, LED_SMD:LED_0603_1608Metric_Pad1.05x0.95mm_HandSolder, F.Cu at (229.4, 79.5)
- added D5: LED_Small_Filled, LED_SMD:LED_0603_1608Metric_Pad1.05x0.95mm_HandSolder, F.Cu at (115.6, 80.0)
- added D50: LED_Small_Filled, LED_SMD:LED_0603_1608Metric_Pad1.05x0.95mm_HandSolder, F.Cu at (232.0, 79.5)
- added D51: LED_Small_Filled, LED_SMD:LED_0603_1608Metric_Pad1.05x0.95mm_HandSolder, F.Cu at (234.6, 79.5)
- added D52: LED_Small_Filled, LED_SMD:LED_0603_1608Metric_Pad1.05x0.95mm_HandSolder, F.Cu at (237.1, 79.5)
- added D53: LED_Small_Filled, LED_SMD:LED_0603_1608Metric_Pad1.05x0.95mm_HandSolder, F.Cu at (239.7, 79.5)
- added D54: LED_Small_Filled, LED_SMD:LED_0603_1608Metric_Pad1.05x0.95mm_HandSolder, F.Cu at (242.3, 79.5)
- added D55: LED_Small_Filled, LED_SMD:LED_0603_1608Metric_Pad1.05x0.95mm_HandSolder, F.Cu at (244.9, 79.5)
- added D56: LED_Small_Filled, LED_SMD:LED_0603_1608Metric_Pad1.05x0.95mm_HandSolder, F.Cu at (247.5, 79.5)
- added D57: LED_Small_Filled, LED_SMD:LED_0603_1608Metric_Pad1.05x0.95mm_HandSolder, F.Cu at (250.1, 79.5)
- added D58: LED_Small_Filled, LED_SMD:LED_0603_1608Metric_Pad1.05x0.95mm_HandSolder, F.Cu at (252.7, 79.5)
- added D59: LED_Small_Filled, LED_SMD:LED_0603_1608Metric_Pad1.05x0.95mm_HandSolder, F.Cu at (255.3, 79.5)
- added D6: LED_Small_Filled, LED_SMD:LED_0603_1608Metric_Pad1.05x0.95mm_HandSolder, F.Cu at (118.1, 80.0)
- added D60: LED_Small_Filled, LED_SMD:LED_0603_1608Metric_Pad1.05x0.95mm_HandSolder, F.Cu at (257.9, 79.5)
- added D61: LED_Small_Filled, LED_SMD:LED_0603_1608Metric_Pad1.05x0.95mm_HandSolder, F.Cu at (224.2, 75.1)
- added D62: LED_Small_Filled, LED_SMD:LED_0603_1608Metric_Pad1.05x0.95mm_HandSolder, F.Cu at (226.8, 75.1)
- added D63: LED_Small_Filled, LED_SMD:LED_0603_1608Metric_Pad1.05x0.95mm_HandSolder, F.Cu at (229.4, 75.1)
- added D64: LED_Small_Filled, LED_SMD:LED_0603_1608Metric_Pad1.05x0.95mm_HandSolder, F.Cu at (232.0, 75.1)
- added D65: LED_Small_Filled, LED_SMD:LED_0603_1608Metric_Pad1.05x0.95mm_HandSolder, F.Cu at (234.6, 75.1)
- added D66: LED_Small_Filled, LED_SMD:LED_0603_1608Metric_Pad1.05x0.95mm_HandSolder, F.Cu at (237.1, 75.1)
- added D67: LED_Small_Filled, LED_SMD:LED_0603_1608Metric_Pad1.05x0.95mm_HandSolder, F.Cu at (239.7, 75.1)
- added D68: LED_Small_Filled, LED_SMD:LED_0603_1608Metric_Pad1.05x0.95mm_HandSolder, F.Cu at (242.3, 75.1)
- added D69: LED_Small_Filled, LED_SMD:LED_0603_1608Metric_Pad1.05x0.95mm_HandSolder, F.Cu at (244.9, 75.1)
- added D7: LED_Small_Filled, LED_SMD:LED_0603_1608Metric_Pad1.05x0.95mm_HandSolder, F.Cu at (120.7, 80.0)
- added D70: LED_Small_Filled, LED_SMD:LED_0603_1608Metric_Pad1.05x0.95mm_HandSolder, F.Cu at (247.5, 75.1)
- added D71: LED_Small_Filled, LED_SMD:LED_0603_1608Metric_Pad1.05x0.95mm_HandSolder, F.Cu at (250.1, 75.1)
- added D72: LED_Small_Filled, LED_SMD:LED_0603_1608Metric_Pad1.05x0.95mm_HandSolder, F.Cu at (252.7, 75.1)
- added D73: LED_Small_Filled, LED_SMD:LED_0603_1608Metric_Pad1.05x0.95mm_HandSolder, F.Cu at (255.3, 75.1)
- added D74: LED_Small_Filled, LED_SMD:LED_0603_1608Metric_Pad1.05x0.95mm_HandSolder, F.Cu at (257.9, 75.1)
- added D75: LED_Small_Filled, LED_SMD:LED_0603_1608Metric_Pad1.05x0.95mm_HandSolder, F.Cu at (224.2, 70.7)
- added D76: LED_Small_Filled, LED_SMD:LED_0603_1608Metric_Pad1.05x0.95mm_HandSolder, F.Cu at (226.8, 70.7)
- added D77: LED_Small_Filled, LED_SMD:LED_0603_1608Metric_Pad1.05x0.95mm_HandSolder, F.Cu at (229.4, 70.7)
- added D78: LED_Small_Filled, LED_SMD:LED_0603_1608Metric_Pad1.05x0.95mm_HandSolder, F.Cu at (232.0, 70.7)
- added D79: LED_Small_Filled, LED_SMD:LED_0603_1608Metric_Pad1.05x0.95mm_HandSolder, F.Cu at (234.6, 70.7)
- added D8: LED_Small_Filled, LED_SMD:LED_0603_1608Metric_Pad1.05x0.95mm_HandSolder, F.Cu at (123.2, 80.0)
- added D80: LED_Small_Filled, LED_SMD:LED_0603_1608Metric_Pad1.05x0.95mm_HandSolder, F.Cu at (237.1, 70.7)
- added D81: LED_Small_Filled, LED_SMD:LED_0603_1608Metric_Pad1.05x0.95mm_HandSolder, F.Cu at (239.7, 70.7)
- added D82: LED_Small_Filled, LED_SMD:LED_0603_1608Metric_Pad1.05x0.95mm_HandSolder, F.Cu at (242.3, 70.7)
- added D83: LED_Small_Filled, LED_SMD:LED_0603_1608Metric_Pad1.05x0.95mm_HandSolder, F.Cu at (244.9, 70.7)
- added D84: LED_Small_Filled, LED_SMD:LED_0603_1608Metric_Pad1.05x0.95mm_HandSolder, F.Cu at (247.5, 70.7)
- added D85: LED_Small_Filled, LED_SMD:LED_0603_1608Metric_Pad1.05x0.95mm_HandSolder, F.Cu at (250.1, 70.7)
- added D86: LED_Small_Filled, LED_SMD:LED_0603_1608Metric_Pad1.05x0.95mm_HandSolder, F.Cu at (252.7, 70.7)
- added D87: LED_Small_Filled, LED_SMD:LED_0603_1608Metric_Pad1.05x0.95mm_HandSolder, F.Cu at (255.3, 70.7)
- added D88: LED_Small_Filled, LED_SMD:LED_0603_1608Metric_Pad1.05x0.95mm_HandSolder, F.Cu at (257.9, 70.7)
- added D89: LED_Small_Filled, LED_SMD:LED_0603_1608Metric_Pad1.05x0.95mm_HandSolder, F.Cu at (224.2, 66.3)
- added D90: LED_Small_Filled, LED_SMD:LED_0603_1608Metric_Pad1.05x0.95mm_HandSolder, F.Cu at (226.8, 66.3)
- added D91: LED_Small_Filled, LED_SMD:LED_0603_1608Metric_Pad1.05x0.95mm_HandSolder, F.Cu at (229.4, 66.3)
- added D92: LED_Small_Filled, LED_SMD:LED_0603_1608Metric_Pad1.05x0.95mm_HandSolder, F.Cu at (232.0, 66.3)
- added D93: LED_Small_Filled, LED_SMD:LED_0603_1608Metric_Pad1.05x0.95mm_HandSolder, F.Cu at (234.6, 66.3)
- added D94: LED_Small_Filled, LED_SMD:LED_0603_1608Metric_Pad1.05x0.95mm_HandSolder, F.Cu at (237.1, 66.3)
- added D95: LED_Small_Filled, LED_SMD:LED_0603_1608Metric_Pad1.05x0.95mm_HandSolder, F.Cu at (239.7, 66.3)
- added D96: LED_Small_Filled, LED_SMD:LED_0603_1608Metric_Pad1.05x0.95mm_HandSolder, F.Cu at (242.3, 66.3)
- added J1: Conn_01x01, Connector_PinSocket_2.54mm:PinSocket_1x01_P2.54mm_Vertical, F.Cu at (170.2, 54.0)
- added J10: Conn_01x04, Connector_PinSocket_2.54mm:PinSocket_1x04_P2.54mm_Vertical, F.Cu at (165.1, 63.5)
- added J11: Conn_01x01, Connector_PinSocket_2.54mm:PinSocket_1x01_P2.54mm_Vertical, F.Cu at (105.4, 59.7)
- added J12: Conn_01x01, Connector_PinSocket_2.54mm:PinSocket_1x01_P2.54mm_Vertical, F.Cu at (108.0, 59.7)
- added J13: Conn_01x01, Connector_PinSocket_2.54mm:PinSocket_1x01_P2.54mm_Vertical, F.Cu at (110.5, 59.7)
- added J14: Conn_01x01, Connector_PinSocket_2.54mm:PinSocket_1x01_P2.54mm_Vertical, F.Cu at (113.0, 59.7)
- added J15: Conn_01x01, Connector_PinSocket_2.54mm:PinSocket_1x01_P2.54mm_Vertical, F.Cu at (115.6, 59.7)
- added J16: Conn_01x01, Connector_PinSocket_2.54mm:PinSocket_1x01_P2.54mm_Vertical, F.Cu at (118.1, 59.7)
- added J17: Conn_01x01, Connector_PinSocket_2.54mm:PinSocket_1x01_P2.54mm_Vertical, F.Cu at (120.7, 59.7)
- added J18: Conn_01x04, Connector_PinSocket_2.54mm:PinSocket_1x04_P2.54mm_Vertical, F.Cu at (177.8, 63.5)
- added J19: Conn_01x01, Connector_PinSocket_2.54mm:PinSocket_1x01_P2.54mm_Vertical, F.Cu at (123.2, 59.7)
- added J20: Conn_02x05_Odd_Even, Connector_PinHeader_2.54mm:PinHeader_2x05_P2.54mm_Vertical, F.Cu at (198.1, 64.8)
- added J21: Conn_01x01, Connector_PinSocket_2.54mm:PinSocket_1x01_P2.54mm_Vertical, F.Cu at (125.7, 59.7)
- added J22: Conn_01x01, Connector_PinSocket_2.54mm:PinSocket_1x01_P2.54mm_Vertical, F.Cu at (128.3, 59.7)
- added J23: Conn_01x01, Connector_PinSocket_2.54mm:PinSocket_1x01_P2.54mm_Vertical, F.Cu at (151.1, 64.8)
- added J24: Conn_01x01, Connector_PinSocket_2.54mm:PinSocket_1x01_P2.54mm_Vertical, F.Cu at (148.6, 64.8)
- added J25: Conn_01x01, Connector_PinSocket_2.54mm:PinSocket_1x01_P2.54mm_Vertical, F.Cu at (146.1, 64.8)
- added J26: Conn_01x01, Connector_PinSocket_2.54mm:PinSocket_1x01_P2.54mm_Vertical, F.Cu at (143.5, 64.8)
- added J27: Conn_01x04, Connector_PinSocket_2.54mm:PinSocket_1x04_P2.54mm_Vertical, F.Cu at (188.0, 63.5)
- added J28: Conn_01x01, Connector_PinSocket_2.54mm:PinSocket_1x01_P2.54mm_Vertical, F.Cu at (141.0, 64.8)
- added J29: Conn_01x01, Connector_PinSocket_2.54mm:PinSocket_1x01_P2.54mm_Vertical, F.Cu at (138.4, 64.8)
- added J30: Conn_02x05_Odd_Even, Connector_PinHeader_2.54mm:PinHeader_2x05_P2.54mm_Vertical, F.Cu at (198.1, 76.2)
- added J31: Conn_01x20, Connector_PinSocket_2.54mm:PinSocket_1x20_P2.54mm_Vertical, F.Cu at (105.4, 74.9)
- added J32: Conn_01x20, Connector_PinSocket_2.54mm:PinSocket_1x20_P2.54mm_Vertical, F.Cu at (105.4, 52.1)
- added J33: Conn_01x20, Connector_PinSocket_2.54mm:PinSocket_1x20_P2.54mm_Vertical, F.Cu at (105.4, 49.5)
- added J6: Conn_01x08, Connector_PinHeader_2.54mm:PinHeader_1x08_P2.54mm_Vertical, F.Cu at (181.6, 48.3)
- added J7: Conn_01x04, Connector_PinSocket_2.54mm:PinSocket_1x04_P2.54mm_Vertical, F.Cu at (205.8, 55.9)
- added J9: Conn_01x04, Connector_PinSocket_2.54mm:PinSocket_1x04_P2.54mm_Vertical, F.Cu at (161.8, 63.5)
- C1, IC1: moved to B.Cu
- J3: value Conn_01x04 -> Conn_01x01; footprint Connector_PinSocket_2.54mm:PinSocket_1x04_P2.54mm_Vertical -> Connector_PinSocket_2.54mm:PinSocket_1x01_P2.54mm_Vertical
- SW10, SW12, SW2, SW4, SW6, SW8: footprint Button_Switch_THT:SW_TH_Tactile_Omron_B3F-110x -> Button_Switch_THT:SW_TH_Tactile_Omron_B3F-100x
- moved D1 155.2 mm to (104.1, 80.0), turned to 90 degrees
- moved D2 152.3 mm to (106.7, 80.0), turned to 90 degrees
- moved D9 131.8 mm to (127.0, 80.0), turned to 90 degrees
- moved D10 128.9 mm to (129.5, 80.0), turned to 90 degrees
- moved RV11 96.4 mm to (144.8, 112.9)
- moved RV12 96.4 mm to (144.8, 112.9)
- moved RV5 89.3 mm to (133.3, 113.0)
- moved RV6 89.3 mm to (133.3, 112.9)
- moved RV13 89.3 mm to (110.5, 113.0)
- moved RV14 89.3 mm to (110.5, 112.9)
- moved RV19 89.3 mm to (121.9, 113.0)
- moved RV20 89.3 mm to (121.9, 112.9)
- moved C1 87.5 mm to (184.2, 95.2), turned to 180 degrees
- moved IC1 54.7 mm to (180.3, 86.4), turned to 90 degrees
- moved U2 54.3 mm to (105.4, 69.8), turned to 90 degrees
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- renumbered A2 to A3, D4 to D10, D3 to D9, J5 to J4, J7 to J5, J1 to J8, RV4 to RV10, RV18 to RV11, RV20 to RV12, RV5 to RV15, RV6 to RV16, RV7 to RV17, RV8 to RV18, RV15 to RV19, RV16 to RV20, RV9 to RV3, RV10 to RV4, RV17 to RV5, RV19 to RV6, RV11 to RV7, RV12 to RV8, RV3 to RV9, U2 to U1, U1 to U2
Connections:
- A1 pad 10: a1 -> Net-(A1-A1)
- A1 pad 11: a2 -> Net-(A1-A2)
- A1 pad 12: a3 -> Net-(A1-A3)
- A1 pad 13: a4 -> Net-(A1-A4)
- A1 pad 14: a5 -> Net-(A1-A5)
- A1 pad 15: unconnected-(A1-D0/RX-Pad15) -> Net-(A1-D0/RX)
- A1 pad 16: unconnected-(A1-D1/TX-Pad16) -> Net-(A1-D1/TX)
- A1 pad 17: I2C_SDA -> Net-(A1-D2/SDA)
- A1 pad 18: I2C_SCL -> Net-(A1-D3/SCL)
- A1 pad 19: sw0 -> Net-(A1-D4)
- A1 pad 2: unconnected-(A1-IOREF-Pad2) -> Net-(A1-IOREF)
- A1 pad 20: sw1 -> Net-(A1-D5)
- A1 pad 21: sw2 -> Net-(A1-D6)
- A1 pad 22: sw3 -> Net-(A1-D7)
- A1 pad 23: sw4 -> Net-(A1-D8)
- A1 pad 24: sw5 -> Net-(A1-D9)
- A1 pad 25: unconnected-(A1-D10-Pad25) -> Net-(A1-D10)
- A1 pad 26: unconnected-(A1-D11-Pad26) -> Net-(A1-D11)
- A1 pad 27: unconnected-(A1-D12-Pad27) -> Net-(A1-D12)
- A1 pad 28: unconnected-(A1-D13-Pad28) -> Net-(A1-D13)
- A1 pad 29: GND -> Net-(A1-GND-Pad29)
- A1 pad 3: unconnected-(A1-~{RESET}-Pad3) -> Net-(A1-~{RESET})
- A1 pad 30: avref -> Net-(A1-AREF)
- A1 pad 31: unconnected-(A1-SDA/D2-Pad31) -> Net-(A1-SDA/D2)
- A1 pad 32: unconnected-(A1-SCL/D3-Pad32) -> Net-(A1-SCL/D3)
- A1 pad 4: +3.3V -> Net-(A1-3V3)
- A1 pad 5: +5VP -> Net-(A1-+5V)
- A1 pad 6: GND -> Net-(A1-GND-Pad6)
- A1 pad 7: GND -> Net-(A1-GND-Pad7)
- A1 pad 8: unconnected-(A1-VIN-Pad8) -> Net-(A1-VIN)
- A1 pad 9: a0 -> Net-(A1-A0)
- A3 pad 10: sw3 -> unconnected-(A3-D7-Pad10)
- A3 pad 11: sw4 -> unconnected-(A3-D8-Pad11)
- A3 pad 12: sw5 -> unconnected-(A3-D9-Pad12)
- A3 pad 18: avref -> unconnected-(A3-AREF-Pad18)
- A3 pad 19: a0 -> unconnected-(A3-A0-Pad19)
- A3 pad 20: a1 -> unconnected-(A3-A1-Pad20)
- A3 pad 21: a2 -> unconnected-(A3-A2-Pad21)
- A3 pad 22: a3 -> unconnected-(A3-A3-Pad22)
- A3 pad 23: a4 -> unconnected-(A3-A4-Pad23)
- A3 pad 24: a5 -> unconnected-(A3-A5-Pad24)
- A3 pad 25: a6 -> unconnected-(A3-A6-Pad25)
- A3 pad 26: a7 -> unconnected-(A3-A7-Pad26)
- A3 pad 29: GND -> unconnected-(A3-GND-Pad29)
- A3 pad 4: GND -> unconnected-(A3-GND-Pad4)
- A3 pad 5: I2C_SDA -> unconnected-(A3-D2-Pad5)
- A3 pad 6: I2C_SCL -> unconnected-(A3-D3-Pad6)
- A3 pad 7: sw0 -> unconnected-(A3-D4-Pad7)
- A3 pad 8: sw1 -> unconnected-(A3-D5-Pad8)
- A3 pad 9: sw2 -> unconnected-(A3-D6-Pad9)
- IC1 pad 10: unconnected-(IC1-ROW11/K10/INT-Pad10) -> Net-(D89-A)
- IC1 pad 11: unconnected-(IC1-ROW10/K9-Pad11) -> Net-(D11-K)
- IC1 pad 12: unconnected-(IC1-ROW9/K8-Pad12) -> Net-(D73-A)
- IC1 pad 13: unconnected-(IC1-ROW8/K7-Pad13) -> Net-(D65-A)
- IC1 pad 14: unconnected-(IC1-ROW7/K6-Pad14) -> Net-(D57-A)
- IC1 pad 15: unconnected-(IC1-ROW6/K5-Pad15) -> Net-(D49-A)
- IC1 pad 16: unconnected-(IC1-ROW5/K4-Pad16) -> Net-(D41-A)
- IC1 pad 17: unconnected-(IC1-ROW4/K3-Pad17) -> Net-(D33-A)
- IC1 pad 18: unconnected-(IC1-ROW3/K2-Pad18) -> Net-(D25-A)
- IC1 pad 19: unconnected-(IC1-ROW2/K1-Pad19) -> Net-(D17-A)
- IC1 pad 4: unconnected-(IC1-COM2/KS1-Pad4) -> Net-(D11-K)
- IC1 pad 5: unconnected-(IC1-COM3/KS2-Pad5) -> Net-(D12-K)
- IC1 pad 6: unconnected-(IC1-COM4-Pad6) -> Net-(D13-K)
- IC1 pad 7: unconnected-(IC1-COM5-Pad7) -> Net-(D14-K)
- IC1 pad 8: unconnected-(IC1-COM6-Pad8) -> Net-(D15-K)
- IC1 pad 9: unconnected-(IC1-COM7-Pad9) -> Net-(D16-K)
- J3 pad 1: Net-(J3-Pin_1) -> Net-(J2-D-)
- J5 pad 1: GND -> Net-(J5-Pin_1)
- J5 pad 2: +3.3V -> Net-(J5-Pin_2)
- J5 pad 3: SPI_SCLK -> Net-(J5-Pin_3)
- J5 pad 4: SPI_MOSI -> Net-(J5-Pin_4)
- J5 pad 5: spi_lcd_res -> Net-(J5-Pin_5)
- J5 pad 6: SPI_MISO -> Net-(J5-Pin_6)
- J5 pad 7: SPI_SS -> Net-(J5-Pin_7)
- J5 pad 8: LCD_BLK -> Net-(J5-Pin_8)
- J8 pad 1: I2C_SCL -> Net-(J7-Pin_1)
- J8 pad 2: I2C_SDA -> Net-(J7-Pin_2)
- J8 pad 3: +3.3V -> Net-(J7-Pin_3)
- J8 pad 4: GND -> Net-(J7-Pin_4)
- RV1 pad 2: a0 -> /pots/a0
- RV10 pad 2: a1 -> /pots/a1
- RV11 pad 2: a9 -> /pots/a9
- RV12 pad 2: a9 -> /pots/a9
- RV13 pad 2: a6 -> /pots/a6
- RV14 pad 2: a6 -> /pots/a6
- RV15 pad 2: a2 -> /pots/a2
- RV16 pad 2: a2 -> /pots/a2
- RV17 pad 2: a3 -> /pots/a3
- RV18 pad 2: a3 -> /pots/a3
- RV19 pad 2: a7 -> /pots/a7
- RV2 pad 2: a0 -> /pots/a0
- RV20 pad 2: a7 -> /pots/a7
- RV3 pad 2: a4 -> /pots/a4
- RV4 pad 2: a4 -> /pots/a4
- RV5 pad 2: a8 -> /pots/a8
- RV6 pad 2: a8 -> /pots/a8
- RV7 pad 2: a5 -> /pots/a5
- RV8 pad 2: a5 -> /pots/a5
- RV9 pad 2: a1 -> /pots/a1
- SW1 pad 1: sw0 -> /pots/sw0
- SW10 pad 1: sw4 -> /pots/sw4
- SW11 pad 1: sw5 -> /pots/sw5
- SW12 pad 1: sw5 -> /pots/sw5
- SW2 pad 1: sw0 -> /pots/sw0
- SW3 pad 1: sw1 -> /pots/sw1
- SW4 pad 1: sw1 -> /pots/sw1
- SW5 pad 1: sw2 -> /pots/sw2
- SW6 pad 1: sw2 -> /pots/sw2
- SW7 pad 1: sw3 -> /pots/sw3
- SW8 pad 1: sw3 -> /pots/sw3
- SW9 pad 1: sw4 -> /pots/sw4
- U1 pad 10: SPI_SS -> unconnected-(U1-PA15-Pad10)
- U1 pad 11: SPI_SCLK -> unconnected-(U1-PB3-Pad11)
- U1 pad 12: SPI_MISO -> unconnected-(U1-PB4-Pad12)
- U1 pad 13: SPI_MOSI -> unconnected-(U1-PB5-Pad13)
- U1 pad 14: I2C_SCL -> unconnected-(U1-PB6-Pad14)
- U1 pad 15: I2C_SDA -> unconnected-(U1-PB7-Pad15)
- U1 pad 17: GND -> unconnected-(U1-GND-Pad17)
- U1 pad 18: GND -> unconnected-(U1-GND-Pad18)
- U1 pad 2: sw3 -> unconnected-(U1-PB13-Pad2)
- U1 pad 23: a0 -> unconnected-(U1-PA0-Pad23)
- U1 pad 24: a1 -> unconnected-(U1-PA1-Pad24)
- U1 pad 25: a2 -> unconnected-(U1-PA2-Pad25)
- U1 pad 26: a3 -> unconnected-(U1-PA3-Pad26)
- U1 pad 27: a4 -> unconnected-(U1-PA4-Pad27)
- U1 pad 28: a5 -> unconnected-(U1-PA5-Pad28)
- U1 pad 29: a6 -> unconnected-(U1-PA6-Pad29)
- U1 pad 3: sw4 -> unconnected-(U1-PB14-Pad3)
- U1 pad 30: a7 -> unconnected-(U1-PA7-Pad30)
- U1 pad 31: a8 -> unconnected-(U1-PB0-Pad31)
- U1 pad 32: a9 -> unconnected-(U1-PB1-Pad32)
- U1 pad 4: sw5 -> unconnected-(U1-PB15-Pad4)
- U1 pad 8: USB_DM -> unconnected-(U1-PA11-Pad8)
- U1 pad 9: USB_DP -> unconnected-(U1-PA12-Pad9)
- U2 pad 10: SPI_SS -> unconnected-(U2-PA15-Pad10)
- U2 pad 11: SPI_SCLK -> unconnected-(U2-PB3-Pad11)
- U2 pad 12: SPI_MISO -> unconnected-(U2-PB4-Pad12)
- U2 pad 13: SPI_MOSI -> unconnected-(U2-PB5-Pad13)
- U2 pad 14: I2C_SCL -> unconnected-(U2-PB6-Pad14)
- U2 pad 15: I2C_SDA -> unconnected-(U2-PB7-Pad15)
- U2 pad 18: +5VP -> unconnected-(U2-5V-Pad18)
- U2 pad 19: GND -> unconnected-(U2-GND-Pad19)
- U2 pad 2: sw3 -> unconnected-(U2-PB13-Pad2)
- U2 pad 20: +3.3V -> unconnected-(U2-3V3-Pad20)
- U2 pad 25: a0 -> unconnected-(U2-PA0-Pad25)
- U2 pad 26: a1 -> unconnected-(U2-PA1-Pad26)
- U2 pad 27: a2 -> unconnected-(U2-PA2-Pad27)
- U2 pad 28: a3 -> unconnected-(U2-PA3-Pad28)
- U2 pad 29: a4 -> unconnected-(U2-PA4-Pad29)
- U2 pad 3: sw4 -> unconnected-(U2-PB14-Pad3)
- U2 pad 30: a5 -> unconnected-(U2-PA5-Pad30)
- U2 pad 31: a6 -> unconnected-(U2-PA6-Pad31)
- U2 pad 32: a7 -> unconnected-(U2-PA7-Pad32)
- U2 pad 33: a8 -> unconnected-(U2-PB0-Pad33)
- U2 pad 34: a9 -> unconnected-(U2-PB1-Pad34)
- U2 pad 38: +3.3V -> unconnected-(U2-3V3-Pad38)
- U2 pad 39: GND -> unconnected-(U2-GND-Pad39)
- U2 pad 4: sw5 -> unconnected-(U2-PB15-Pad4)
- U2 pad 40: GND -> unconnected-(U2-GND-Pad40)
- U2 pad 8: USB_DM -> unconnected-(U2-PA11-Pad8)
- U2 pad 9: USB_DP -> unconnected-(U2-PA12-Pad9)
Routing:
- net sw5: track 117.4 -> 0.00 mm
- net sw4: track 96.7 -> 0.00 mm
- net SPI_MOSI: track 75.4 -> 0.00 mm
- net sw3: track 72.9 -> 0.00 mm
- net SPI_MISO: track 72.2 -> 0.00 mm
- net SPI_SCLK: track 67.3 -> 0.00 mm
- net a4: track 65.2 -> 0.00 mm
- net Net-(D10-A): track 0.00 -> 61.7 mm, vias 0 -> 1
- net /pots/a6: track 0.00 -> 61.1 mm
- net /pots/a5: track 0.00 -> 60.5 mm
- net sw1: track 60.5 -> 0.00 mm
- net /pots/a9: track 0.00 -> 59.4 mm
- net a9: track 57.0 -> 0.00 mm
- net /pots/a7: track 0.00 -> 57.0 mm
- net /pots/a8: track 0.00 -> 55.8 mm
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
Commit message: 更新
Parts:
- added D100: LED_Small_Filled, LED_SMD:LED_0603_1608Metric_Pad1.05x0.95mm_HandSolder, F.Cu at (209.7, 88.9)
- added D97: LED_Small_Filled, LED_SMD:LED_0603_1608Metric_Pad1.05x0.95mm_HandSolder, F.Cu at (201.9, 88.9)
- added D98: LED_Small_Filled, LED_SMD:LED_0603_1608Metric_Pad1.05x0.95mm_HandSolder, F.Cu at (204.5, 88.9)
- added D99: LED_Small_Filled, LED_SMD:LED_0603_1608Metric_Pad1.05x0.95mm_HandSolder, F.Cu at (207.1, 88.9)
- added J34: Conn_01x01, Connector_PinSocket_2.54mm:PinSocket_1x01_P2.54mm_Vertical, F.Cu at (133.3, 59.7)
- added J35: Conn_01x04, Connector_PinSocket_2.54mm:PinSocket_1x04_P2.54mm_Vertical, F.Cu at (143.5, 59.7)
- added R1: R_Small_US, Resistor_SMD:R_0402_1005Metric_Pad0.72x0.64mm_HandSolder, F.Cu at (201.9, 85.1)
- added R2: R_Small_US, Resistor_SMD:R_0402_1005Metric_Pad0.72x0.64mm_HandSolder, F.Cu at (204.5, 85.1)
- added R3: R_Small_US, Resistor_SMD:R_0402_1005Metric_Pad0.72x0.64mm_HandSolder, F.Cu at (207.0, 85.1)
- added R4: R_Small_US, Resistor_SMD:R_0402_1005Metric_Pad0.72x0.64mm_HandSolder, F.Cu at (209.6, 85.1)
- moved D74 101.0 mm to (161.4, 105.0)
- moved D73 101.0 mm to (158.8, 105.0)
- moved D57 96.3 mm to (158.7, 110.0)
- moved D58 96.3 mm to (161.3, 110.0)
- moved D59 96.1 mm to (164.3, 110.5)
- moved D60 96.1 mm to (166.9, 110.5)
- moved D44 90.5 mm to (167.6, 116.0)
- moved D45 90.5 mm to (170.2, 116.0)
- moved D46 90.5 mm to (172.8, 116.0)
- moved D41 90.5 mm to (158.8, 116.0)
- moved D42 90.5 mm to (161.3, 116.0)
- moved D43 90.5 mm to (165.1, 116.0)
- moved D76 68.4 mm to (167.1, 104.1)
- moved D77 68.4 mm to (169.7, 104.1)
- moved D78 68.4 mm to (172.3, 104.1)
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