File: jhl_synth0.kicad_pcb (KiCad board)
At the start: 4 copper layers, 178 parts, among them IC1 HT16K33, J1 Conn_01x01, J10 Conn_01x04, J11 Conn_01x01, J12 Conn_01x01, J13 Conn_01x01, J14 Conn_01x01, J15 Conn_01x01, J16 Conn_01x01, J17 Conn_01x01, J18 Conn_01x04, J19 Conn_01x01, J2 USB_B_Micro, J20 Conn_02x05_Odd_Even, J21 Conn_01x01, J22 Conn_01x01, J23 Conn_01x01, J24 Conn_01x01, J25 Conn_01x01, J26 Conn_01x01, J27 Conn_01x04, J28 Conn_01x01, J29 Conn_01x01, J3 Conn_01x01, J30 Conn_02x05_Odd_Even, J31 Conn_01x20, J32 Conn_01x20, J33 Conn_01x20, J34 Conn_01x01, J35 Conn_01x04, J4 Conn_01x01, J5 Conn_01x08, J6 Conn_01x08, J7 Conn_01x04, J8 Conn_01x04, J9 Conn_01x04, SW1 SW_SPST, SW10 SW_SPST, SW11 SW_SPST, SW12 SW_SPST, SW2 SW_SPST, SW3 SW_SPST, SW4 SW_SPST, SW5 SW_SPST, SW6 SW_SPST, SW7 SW_SPST, SW8 SW_SPST, SW9 SW_SPST, U1 YAAJ_BlackPill, U2 YAAJ_BluePill

Commit message: 更新
Parts:
- added D101: ~, libs:BU5004, F.Cu at (199.4, 113.0)
- added R5: R_Small_US, Resistor_SMD:R_0402_1005Metric_Pad0.72x0.64mm_HandSolder, F.Cu at (177.8, 100.3)
- added REF**: PinSocket_1x04_P2.54mm_Vertical, Connector_PinSocket_2.54mm:PinSocket_1x04_P2.54mm_Vertical, F.Cu at (182.9, 100.3)
- added REF**: MountingHole_3.2mm_M3, MountingHole:MountingHole_3.2mm_M3, F.Cu at (199.4, 57.1)
- added REF**: MountingHole_3.2mm_M3, MountingHole:MountingHole_3.2mm_M3, F.Cu at (106.7, 133.3)
- added REF**: MountingHole_3.2mm_M3, MountingHole:MountingHole_3.2mm_M3, F.Cu at (106.7, 64.8)
- added REF**: MountingHole_3.2mm_M3, MountingHole:MountingHole_3.2mm_M3, F.Cu at (207.0, 133.3)
- added REF**: PinSocket_1x04_P2.54mm_Vertical, Connector_PinSocket_2.54mm:PinSocket_1x04_P2.54mm_Vertical, F.Cu at (172.7, 100.3)
- added SW13: SW_SPST, Button_Switch_SMD:SW_Push_1P1T_XKB_TS-1187A, F.Cu at (142.2, 121.9)
- added SW14: SW_SPST, Button_Switch_THT:SW_TH_Tactile_Omron_B3F-100x, F.Cu at (139.0, 119.7)
- added SW15: SW_SPST, Button_Switch_SMD:SW_Push_1P1T_XKB_TS-1187A, F.Cu at (130.8, 121.9)
- added SW16: SW_SPST, Button_Switch_THT:SW_TH_Tactile_Omron_B3F-100x, F.Cu at (127.6, 119.7)
- added SW17: SW_SPST, Button_Switch_SMD:SW_Push_1P1T_XKB_TS-1187A, F.Cu at (119.4, 121.9)
- added SW18: SW_SPST, Button_Switch_THT:SW_TH_Tactile_Omron_B3F-100x, F.Cu at (116.1, 119.7)
- added SW19: SW_SPST, Button_Switch_SMD:SW_Push_1P1T_XKB_TS-1187A, F.Cu at (107.3, 121.9)
- added SW20: SW_SPST, Button_Switch_THT:SW_TH_Tactile_Omron_B3F-100x, F.Cu at (104.1, 119.7)
- added U3: SA39-12SRWA, Display_7Segment:Sx39-1xxxxx, F.Cu at (164.0, 113.2)
- added U4: SA39-12SRWA, Display_7Segment:Sx39-1xxxxx, F.Cu at (151.3, 113.2)
- added U5: PCA9306DC, Package_SO:VSSOP-8_2.3x2mm_P0.5mm, F.Cu at (177.8, 102.9)
- added U6: PCA9306DP, Package_SO:TSSOP-8_3x3mm_P0.65mm, F.Cu at (177.8, 106.7)
- added U7: SA39-12SRWA, Display_7Segment:Sx39-1xxxxx, F.Cu at (176.7, 113.2)
- C1, IC1: moved to F.Cu
- moved D96 130.8 mm to (130.8, 134.6), turned to -90 degrees
- moved D95 130.7 mm to (128.3, 134.6), turned to -90 degrees
- moved D94 130.7 mm to (125.7, 134.6), turned to -90 degrees
- moved D93 130.6 mm to (123.2, 134.6), turned to -90 degrees
- moved D92 130.6 mm to (120.7, 134.6), turned to -90 degrees
- moved D91 130.5 mm to (118.1, 134.6), turned to -90 degrees
- moved D90 130.5 mm to (115.6, 134.6), turned to -90 degrees
- moved D89 130.5 mm to (113.0, 134.6), turned to -90 degrees
- moved D88 71.6 mm to (130.9, 128.3)
- moved D87 71.5 mm to (128.3, 128.3)
- moved D86 71.5 mm to (125.8, 128.3)
- moved D85 71.4 mm to (123.2, 128.3)
- moved D84 71.4 mm to (120.7, 128.3)
- moved D83 71.3 mm to (118.2, 128.3)
- moved D81 71.3 mm to (113.0, 128.3)
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Connections:
- net Net-(D1-A) renamed LED_R0
- net Net-(D1-K) renamed LED_C0
- net Net-(D10-A) renamed LED_R1
- net Net-(D10-K) renamed LED_C1
- net Net-(D12-K) renamed LED_C3
- net Net-(D13-K) renamed LED_C4
- net Net-(D14-K) renamed LED_C5
- net Net-(D15-K) renamed LED_C6
- net Net-(D16-K) renamed LED_C7
- net Net-(D17-A) renamed LED_R2
- net Net-(D25-A) renamed LED_R3
- net Net-(D33-A) renamed LED_R4
- net Net-(D41-A) renamed LED_R5
- net Net-(D49-A) renamed LED_R6
- net Net-(D57-A) renamed LED_R7
- net Net-(D65-A) renamed LED_R8
- net Net-(D73-A) renamed LED_R9
- net Net-(D89-A) renamed LED_R11
- C1 pad 1: +3.3V -> +5VP
- D11 pad 1: Net-(D11-K) -> LED_C2
- D19 pad 1: Net-(D11-K) -> LED_C2
- D27 pad 1: Net-(D11-K) -> LED_C2
- D3 pad 1: Net-(D11-K) -> LED_C2
- D35 pad 1: Net-(D11-K) -> LED_C2
- D43 pad 1: Net-(D11-K) -> LED_C2
- D51 pad 1: Net-(D11-K) -> LED_C2
- D59 pad 1: Net-(D11-K) -> LED_C2
- D67 pad 1: Net-(D11-K) -> LED_C2
- D75 pad 1: Net-(D11-K) -> LED_C2
- D81 pad 2: Net-(D11-K) -> LED_R10
- D82 pad 2: Net-(D11-K) -> LED_R10
- D83 pad 1: Net-(D11-K) -> LED_C2
- D83 pad 2: Net-(D11-K) -> LED_R10
- D84 pad 2: Net-(D11-K) -> LED_R10
- D85 pad 2: Net-(D11-K) -> LED_R10
- D86 pad 2: Net-(D11-K) -> LED_R10
- D87 pad 2: Net-(D11-K) -> LED_R10
- D88 pad 2: Net-(D11-K) -> LED_R10
- D91 pad 1: Net-(D11-K) -> LED_C2
- IC1 pad 11: Net-(D11-K) -> LED_R10
- IC1 pad 24: +3.3V -> +5VP
- IC1 pad 4: Net-(D11-K) -> LED_C2
Routing:
- net LED_C0: track 28.7 -> 157.2 mm, vias 0 -> 4
- net LED_C2: track 0.00 -> 127.3 mm, vias 0 -> 6
- net LED_R9: track 0.00 -> 107.8 mm, vias 0 -> 2
- net LED_C6: track 0.00 -> 98.2 mm, vias 0 -> 2
- net LED_C1: track 0.00 -> 98.0 mm, vias 0 -> 3
- net LED_C7: track 29.8 -> 124.9 mm, vias 0 -> 3
- net LED_C4: track 0.00 -> 88.4 mm, vias 0 -> 4
- net LED_C5: track 0.00 -> 86.6 mm, vias 0 -> 3
- net LED_C3: track 23.5 -> 108.6 mm, vias 0 -> 5
- net /pots/sw0: track 36.6 -> 105.8 mm, vias 0 -> 2
- net LED_R11: track 0.00 -> 67.2 mm, vias 0 -> 1
- net LED_R5: track 0.00 -> 62.9 mm, vias 0 -> 1
- net LED_R10: track 0.00 -> 59.6 mm
- net LED_R7: track 0.00 -> 54.9 mm
- net /pots/sw3: track 40.9 -> 82.2 mm, vias 0 -> 1
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
Commit message: 更新
Parts:
- moved C1 12.6 mm to (189.1, 94.2), turned to 90 degrees
- moved REF** 9.35 mm to (205.7, 64.0)
- moved IC1 4.07 mm to (180.2, 90.4), turned to 180 degrees
Routing:
- net LED_C4: track 88.4 -> 303.1 mm, vias 4 -> 11
- net LED_C1: track 98.0 -> 309.3 mm, vias 3 -> 11
- net LED_C3: track 108.6 -> 318.1 mm, vias 5 -> 11
- net LED_C5: track 86.6 -> 282.7 mm, vias 3 -> 10
- net LED_C2: track 127.3 -> 308.3 mm, vias 6 -> 11
- net LED_C6: track 98.2 -> 274.0 mm, vias 2 -> 10
- net LED_C0: track 157.2 -> 327.4 mm, vias 4 -> 9
- net LED_C7: track 124.9 -> 260.6 mm, vias 3 -> 9
- net LED_R0: track 21.1 -> 149.0 mm, vias 2 -> 4
- net +5VP: track 36.8 -> 148.1 mm, vias 0 -> 2
- net LED_R3: track 19.8 -> 118.0 mm, vias 2 -> 3
- net +3.3V: track 61.9 -> 154.5 mm, vias 1 -> 2
- net LED_R4: track 28.5 -> 117.1 mm, vias 2 -> 3
- net LED_R6: track 17.8 -> 95.5 mm, vias 0 -> 3
- net LED_R1: track 57.5 -> 130.0 mm, vias 4 -> 5
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