File: jhl_synth0.kicad_pcb (KiCad board)
At the start: 4 copper layers, 199 parts, among them IC1 HT16K33, J1 Conn_01x01, J10 Conn_01x04, J11 Conn_01x01, J12 Conn_01x01, J13 Conn_01x01, J14 Conn_01x01, J15 Conn_01x01, J16 Conn_01x01, J17 Conn_01x01, J18 Conn_01x04, J19 Conn_01x01, J2 USB_B_Micro, J20 Conn_02x05_Odd_Even, J21 Conn_01x01, J22 Conn_01x01, J23 Conn_01x01, J24 Conn_01x01, J25 Conn_01x01, J26 Conn_01x01, J27 Conn_01x04, J28 Conn_01x01, J29 Conn_01x01, J3 Conn_01x01, J30 Conn_02x05_Odd_Even, J31 Conn_01x20, J32 Conn_01x20, J33 Conn_01x20, J34 Conn_01x01, J35 Conn_01x04, J4 Conn_01x01, J5 Conn_01x08, J6 Conn_01x08, J7 Conn_01x04, J8 Conn_01x04, J9 Conn_01x04, SW1 SW_SPST, SW10 SW_SPST, SW11 SW_SPST, SW12 SW_SPST, SW13 SW_SPST, SW14 SW_SPST, SW15 SW_SPST, SW16 SW_SPST, SW17 SW_SPST, SW18 SW_SPST, SW19 SW_SPST, SW2 SW_SPST, SW20 SW_SPST, SW3 SW_SPST, SW4 SW_SPST, SW5 SW_SPST, SW6 SW_SPST, SW7 SW_SPST, SW8 SW_SPST, SW9 SW_SPST, U1 YAAJ_BlackPill, U2 YAAJ_BluePill, U3 SA39-12SRWA, U4 SA39-12SRWA, U5 PCA9306DC, U6 PCA9306DP, U7 SA39-12SRWA

Commit message: 更新
Parts:
- added J36: Conn_01x03, Connector_PinHeader_2.54mm:PinHeader_1x03_P2.54mm_Vertical, F.Cu at (153.7, 72.4)
Routing:
- net +3.3V: track 154.5 -> 61.9 mm, vias 2 -> 1
- net +5VP: track 148.1 -> 101.6 mm, vias 2 -> 1
- net I2C_SDA: track 71.8 -> 66.2 mm
- net I2C_SCL: track 80.8 -> 76.5 mm
- net LED_C4: track 303.1 -> 306.7 mm, vias 11 -> 10
- net LED_C0: track 327.4 -> 323.9 mm
- net LED_R7: track 94.6 -> 92.0 mm, vias 1 -> 0
- net GND: track 39.9 -> 41.4 mm
- net LED_R4: track 117.1 -> 116.1 mm
- net LED_R1: track 130.0 -> 130.5 mm
Other:
- board outline added: 111.1 x 92.7 mm

Commit message: 更新
Parts:
- removed A1, A2: Arduino_Leonardo, Module:Arduino_UNO_R3
- removed A3: Arduino_Nano_v3.x, Module:Arduino_Nano
- removed REF** (x2): PinSocket_1x04_P2.54mm_Vertical, Connector_PinSocket_2.54mm:PinSocket_1x04_P2.54mm_Vertical
- removed REF** (x4): MountingHole_3.2mm_M3, MountingHole:MountingHole_3.2mm_M3
- removed U1: YAAJ_BlackPill, libs:YAAJ_BlackPill_1
- removed U2: YAAJ_BluePill, libs:YAAJ_BluePill_1
- added J37: Conn_01x20, Connector_PinSocket_2.54mm:PinSocket_1x20_P2.54mm_Vertical, F.Cu at (105.4, 54.6)
- added J38: Conn_01x20, Connector_PinSocket_2.54mm:PinSocket_1x20_P2.54mm_Vertical, F.Cu at (105.4, 72.4)
- added J39: Conn_01x20, Connector_PinSocket_2.54mm:PinSocket_1x20_P2.54mm_Vertical, F.Cu at (105.4, 69.8)
- added J40: Conn_01x04, Connector_PinSocket_2.54mm:PinSocket_1x04_P2.54mm_Vertical, F.Cu at (182.9, 107.9)
- added J41: Conn_01x10, Connector_PinSocket_2.54mm:PinSocket_1x10_P2.54mm_Vertical, F.Cu at (109.0, 102.9)
- added J42: Conn_01x08, Connector_PinSocket_2.54mm:PinSocket_1x08_P2.54mm_Vertical, F.Cu at (135.9, 102.9)
- added J43: Conn_01x08, Connector_PinSocket_2.54mm:PinSocket_1x08_P2.54mm_Vertical, F.Cu at (135.9, 100.3)
- added J44: Conn_01x10, Connector_PinSocket_2.54mm:PinSocket_1x10_P2.54mm_Vertical, F.Cu at (109.0, 100.3)
- J36: value Conn_01x03 -> Conn_01x04; footprint Connector_PinHeader_2.54mm:PinHeader_1x03_P2.54mm_Vertical -> Connector_PinSocket_2.54mm:PinSocket_1x04_P2.54mm_Vertical
- R1, R2, R3, R4: value R_Small_US -> 1k
- R5: value R_Small_US -> 200k
- moved J36 33.8 mm to (172.7, 100.3), turned to 0 degrees
Connections:
- J31 pad 1: unconnected-(J31-Pin_1-Pad1) -> Net-(J31-Pin_1)
- J31 pad 10: unconnected-(J31-Pin_10-Pad10) -> Net-(J31-Pin_10)
- J31 pad 11: unconnected-(J31-Pin_11-Pad11) -> Net-(J31-Pin_11)
- J31 pad 12: unconnected-(J31-Pin_12-Pad12) -> Net-(J31-Pin_12)
- J31 pad 13: unconnected-(J31-Pin_13-Pad13) -> Net-(J31-Pin_13)
- J31 pad 14: unconnected-(J31-Pin_14-Pad14) -> Net-(J31-Pin_14)
- J31 pad 15: unconnected-(J31-Pin_15-Pad15) -> Net-(J31-Pin_15)
- J31 pad 16: unconnected-(J31-Pin_16-Pad16) -> Net-(J31-Pin_16)
- J31 pad 17: unconnected-(J31-Pin_17-Pad17) -> Net-(J31-Pin_17)
- J31 pad 18: unconnected-(J31-Pin_18-Pad18) -> Net-(J31-Pin_18)
- J31 pad 19: unconnected-(J31-Pin_19-Pad19) -> Net-(J31-Pin_19)
- J31 pad 2: unconnected-(J31-Pin_2-Pad2) -> Net-(J31-Pin_2)
- J31 pad 20: unconnected-(J31-Pin_20-Pad20) -> Net-(J31-Pin_20)
- J31 pad 3: unconnected-(J31-Pin_3-Pad3) -> Net-(J31-Pin_3)
- J31 pad 4: unconnected-(J31-Pin_4-Pad4) -> Net-(J31-Pin_4)
- J31 pad 5: unconnected-(J31-Pin_5-Pad5) -> Net-(J31-Pin_5)
- J31 pad 6: unconnected-(J31-Pin_6-Pad6) -> Net-(J31-Pin_6)
- J31 pad 7: unconnected-(J31-Pin_7-Pad7) -> Net-(J31-Pin_7)
- J31 pad 8: unconnected-(J31-Pin_8-Pad8) -> Net-(J31-Pin_8)
- J31 pad 9: unconnected-(J31-Pin_9-Pad9) -> Net-(J31-Pin_9)
- J36 pad 1: unconnected-(J36-Pin_1-Pad1) -> +3.3V
- J36 pad 2: unconnected-(J36-Pin_2-Pad2) -> I2C_SCL
- J36 pad 3: unconnected-(J36-Pin_3-Pad3) -> I2C_SDA
Routing:
- net Net-(J31-Pin_9): track 0.00 -> 5.08 mm
- net Net-(J31-Pin_8): track 0.00 -> 5.08 mm
- net Net-(J31-Pin_7): track 0.00 -> 5.08 mm
- net Net-(J31-Pin_6): track 0.00 -> 5.08 mm
- net Net-(J31-Pin_5): track 0.00 -> 5.08 mm
- net Net-(J31-Pin_4): track 0.00 -> 5.08 mm
- net Net-(J31-Pin_3): track 0.00 -> 5.08 mm
- net Net-(J31-Pin_20): track 0.00 -> 5.08 mm
- net Net-(J31-Pin_2): track 0.00 -> 5.08 mm
- net Net-(J31-Pin_19): track 0.00 -> 5.08 mm
- net Net-(J31-Pin_18): track 0.00 -> 5.08 mm
- net Net-(J31-Pin_17): track 0.00 -> 5.08 mm
- net Net-(J31-Pin_16): track 0.00 -> 5.08 mm
- net Net-(J31-Pin_15): track 0.00 -> 5.08 mm
- net Net-(J31-Pin_14): track 0.00 -> 5.08 mm
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Other:
- board text added: "Molex-105017-0001"

Commit message: 更新
Parts:
- added H1: MountingHole, MountingHole:MountingHole_3.2mm_M3, F.Cu at (207.0, 63.5)
- added H2: MountingHole, MountingHole:MountingHole_3.2mm_M3, F.Cu at (207.0, 132.7)
- added H3: MountingHole, MountingHole:MountingHole_3.2mm_M3, F.Cu at (106.7, 132.7)
- added H4: MountingHole, MountingHole:MountingHole_3.2mm_M3, F.Cu at (106.0, 64.8)
- added J45: Conn_01x01, Connector_PinSocket_2.54mm:PinSocket_1x01_P2.54mm_Vertical, F.Cu at (143.5, 64.8)
- added J46: Conn_01x01, Connector_PinSocket_2.54mm:PinSocket_1x01_P2.54mm_Vertical, F.Cu at (146.1, 64.8)
- added J47: Conn_01x01, Connector_PinSocket_2.54mm:PinSocket_1x01_P2.54mm_Vertical, F.Cu at (148.6, 64.8)
- added J48: Conn_01x01, Connector_PinSocket_2.54mm:PinSocket_1x01_P2.54mm_Vertical, F.Cu at (151.1, 64.8)
- moved SW1 57.1 mm to (108.0, 94.0)
- moved SW11 57.1 mm to (165.1, 94.0)
- moved SW12 57.1 mm to (161.8, 91.7)
- moved SW2 57.1 mm to (104.7, 91.7)
- moved SW13 34.9 mm to (107.3, 121.9)
- moved SW14 34.9 mm to (104.1, 119.7)
- moved SW19 34.9 mm to (142.2, 121.9)
- moved SW20 34.9 mm to (139.0, 119.7)
- moved SW10 34.3 mm to (150.4, 91.7)
- moved SW3 34.3 mm to (119.4, 94.0)
- moved SW4 34.3 mm to (116.1, 91.7)
- moved SW9 34.3 mm to (153.7, 94.0)
- moved J23 22.9 mm to (128.3, 64.8), turned to 0 degrees
- moved J24 17.8 mm to (130.8, 64.8), turned to 0 degrees
- moved J25 12.7 mm to (133.3, 64.8), turned to 0 degrees
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Connections:
- SW13 pad 1: /pots/sw0 -> /pots/sw6
- SW14 pad 1: /pots/sw0 -> /pots/sw6
- SW15 pad 1: /pots/sw1 -> /pots/sw7
- SW16 pad 1: /pots/sw1 -> /pots/sw7
- SW17 pad 1: /pots/sw2 -> /pots/sw8
- SW18 pad 1: /pots/sw2 -> /pots/sw8
- SW19 pad 1: /pots/sw3 -> /pots/sw9
- SW20 pad 1: /pots/sw3 -> /pots/sw9
Routing:
- net /pots/sw6: track 0.00 -> 86.2 mm
- net /pots/sw7: track 0.00 -> 71.7 mm
- net /pots/sw8: track 0.00 -> 65.0 mm
- net /pots/sw9: track 0.00 -> 57.2 mm
- net /pots/sw2: track 72.9 -> 28.5 mm
- net /pots/sw3: track 72.8 -> 28.6 mm, vias 1 -> 0
- net /pots/sw1: track 67.8 -> 30.3 mm
- net /pots/sw0: track 70.8 -> 37.9 mm, vias 2 -> 0
- net LED_C2: track 308.2 -> 337.8 mm
- net GND: track 41.4 -> 18.5 mm
- net unconnected-(J2-Shield-Pad6): track 0.00 -> 11.5 mm
- net /pots/sw5: track 50.1 -> 41.5 mm
- net LED_R1: track 129.2 -> 136.9 mm, vias 5 -> 10
- net /pots/sw4: track 39.5 -> 32.3 mm
- net LED_R7: track 92.0 -> 86.6 mm, vias 0 -> 1
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Other:
- board text added: "+3.3 GND"
- board text added: "0 1 2 3 4 5 6 7 0 1 2 3 4 5 6 7 0 1 2 3 4 5 6 7 0 1 2 3 4 5 6 7"
- board text added: "1"
- board text added: "1 2"
- board text added: "17"
- board text added: "3 4"
- board text added: "5 6"
- board text added: "7 8"
- board text added: "9"
- board text added: "9 10"
- board text added: "A K"
- board text added: "A0 v5 10"
- board text added: "AVref"
- board text added: "I2C SCL SDA"
- board text added: "I2C for LCD"
- board text added: "ID D+ D-"
- board text added: "K A"
- board text added: "LED 1 2 3 4"
- board text added: "LED 1..4"
- board text added: "R10"
- board text added: "R11"
- board text added: "R5"
- board text added: "R6"
- board text added: "R7"
- board text added: "R8"
- board text added: "R9"
- board text added: "SW 1..10"
- board text added: "[GROVE] GND Vcc SDA SCL"
