File: jhl_synth0.kicad_pcb (KiCad board)
At the start: 4 copper layers, 111.1 x 92.7 mm, 205 parts, among them IC1 HT16K33, J1 Conn_01x01, J10 Conn_01x04, J11 Conn_01x01, J12 Conn_01x01, J13 Conn_01x01, J14 Conn_01x01, J15 Conn_01x01, J16 Conn_01x01, J17 Conn_01x01, J18 Conn_01x04, J19 Conn_01x01, J2 USB_B_Micro, J20 Conn_02x05_Odd_Even, J21 Conn_01x01, J22 Conn_01x01, J23 Conn_01x01, J24 Conn_01x01, J25 Conn_01x01, J26 Conn_01x01, J27 Conn_01x04, J28 Conn_01x01, J29 Conn_01x01, J3 Conn_01x01, J30 Conn_02x05_Odd_Even, J31 Conn_01x20, J32 Conn_01x20, J33 Conn_01x20, J34 Conn_01x01, J35 Conn_01x04, J36 Conn_01x04, J37 Conn_01x20, J38 Conn_01x20, J39 Conn_01x20, J4 Conn_01x01, J40 Conn_01x04, J41 Conn_01x10, J42 Conn_01x08, J43 Conn_01x08, J44 Conn_01x10, J45 Conn_01x01, J46 Conn_01x01, J47 Conn_01x01, J48 Conn_01x01, J5 Conn_01x08, J6 Conn_01x08, J7 Conn_01x04, J8 Conn_01x04, J9 Conn_01x04, SW1 SW_SPST, SW10 SW_SPST, SW11 SW_SPST, SW12 SW_SPST, SW13 SW_SPST, SW14 SW_SPST, SW15 SW_SPST, SW16 SW_SPST, SW17 SW_SPST, SW18 SW_SPST, SW19 SW_SPST, SW2 SW_SPST, SW20 SW_SPST, SW3 SW_SPST, SW4 SW_SPST, SW5 SW_SPST, SW6 SW_SPST, SW7 SW_SPST, SW8 SW_SPST, SW9 SW_SPST, U3 SA39-12SRWA, U4 SA39-12SRWA, U5 PCA9306DC, U6 PCA9306DP, U7 SA39-12SRWA

Commit message: 更新
Parts:
- added J49: Conn_01x02, Connector_PinHeader_2.54mm:PinHeader_2x01_P2.54mm_Vertical, F.Cu at (186.7, 128.8)
- added J51: Conn_01x08, Connector_PinHeader_2.54mm:PinHeader_1x08_P2.54mm_Vertical, F.Cu at (159.9, 71.6)
- added J52: Conn_01x04, Connector_PinSocket_2.54mm:PinSocket_1x04_P2.54mm_Vertical, F.Cu at (184.0, 64.0)
- added J53: Conn_02x08_Odd_Even, Connector_PinHeader_2.54mm:PinHeader_2x08_P2.54mm_Vertical, F.Cu at (159.9, 66.5)
- added R10: 200k, Resistor_SMD:R_0402_1005Metric_Pad0.72x0.64mm_HandSolder, F.Cu at (170.1, 69.1)
- added R11: 200k, Resistor_SMD:R_0402_1005Metric_Pad0.72x0.64mm_HandSolder, F.Cu at (172.6, 69.1)
- added R12: 200k, Resistor_SMD:R_0402_1005Metric_Pad0.72x0.64mm_HandSolder, F.Cu at (175.1, 69.1)
- added R13: 200k, Resistor_SMD:R_0402_1005Metric_Pad0.72x0.64mm_HandSolder, F.Cu at (177.7, 69.1)
- added R6: 200k, Resistor_SMD:R_0402_1005Metric_Pad0.72x0.64mm_HandSolder, F.Cu at (159.9, 69.1)
- added R7: 200k, Resistor_SMD:R_0402_1005Metric_Pad0.72x0.64mm_HandSolder, F.Cu at (162.4, 69.1)
- added R8: 200k, Resistor_SMD:R_0402_1005Metric_Pad0.72x0.64mm_HandSolder, F.Cu at (165.0, 69.1)
- added R9: 200k, Resistor_SMD:R_0402_1005Metric_Pad0.72x0.64mm_HandSolder, F.Cu at (167.5, 69.1)
- added U8: PCA9306D, Package_SO:SO-8_3.9x4.9mm_P1.27mm, F.Cu at (164.3, 90.7)
- J2: footprint Connector_USB:USB_Micro-B_Molex-105017-0001 -> libs:usb b micro jhl
- J36, J40: value Conn_01x04 -> Conn_01x02; footprint Connector_PinSocket_2.54mm:PinSocket_1x04_P2.54mm_Vertical -> Connector_PinHeader_2.54mm:PinHeader_2x01_P2.54mm_Vertical
- U5, U6: moved to B.Cu
- moved D42 79.1 mm to (148.6, 49.5)
- moved D43 79.1 mm to (151.1, 49.5)
- moved D44 79.1 mm to (153.7, 49.5)
- moved D45 79.1 mm to (156.2, 49.5)
- moved D46 79.1 mm to (158.8, 49.5)
- moved D47 79.1 mm to (161.3, 49.5)
- moved D49 79.1 mm to (125.7, 49.5)
- moved D51 79.1 mm to (130.8, 49.5)
- moved D52 79.1 mm to (133.3, 49.5)
- moved D53 79.1 mm to (135.9, 49.5)
- moved D54 79.1 mm to (138.4, 49.5)
- moved D55 79.1 mm to (141.0, 49.5)
- moved D56 79.1 mm to (143.5, 49.5)
- moved D57 79.1 mm to (166.4, 55.9)
- moved D58 79.1 mm to (168.9, 55.9)
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Connections:
- IC1 pad 22: I2C_SCL -> I2C_SCL5
- IC1 pad 23: I2C_SDA -> I2C_SDA5
- J36 pad 1: +3.3V -> LED_R8
- J36 pad 2: I2C_SCL -> Net-(J36-Pin_2)
- J40 pad 1: GND -> LED_R9
- J40 pad 2: I2C_SDA5 -> Net-(J40-Pin_2)
- U3 pad 1: LED_R9 -> Net-(J40-Pin_2)
- U3 pad 6: LED_R9 -> Net-(J40-Pin_2)
- U4 pad 1: LED_R8 -> Net-(J36-Pin_2)
- U4 pad 6: LED_R8 -> Net-(J36-Pin_2)
- U7 pad 1: LED_R10 -> Net-(J49-Pin_2)
- U7 pad 6: LED_R10 -> Net-(J49-Pin_2)
Routing:
- net (no net): track 0.00 -> 173.4 mm
- net LED_R3: track 117.4 -> 44.9 mm, vias 3 -> 2
- net +5VP: track 102.4 -> 43.4 mm, vias 1 -> 2
- net LED_R8: track 78.7 -> 136.8 mm, vias 1 -> 3
- net I2C_SCL: track 76.5 -> 19.2 mm
- net LED_C7: track 259.7 -> 315.8 mm, vias 9 -> 10
- net I2C_SDA: track 66.2 -> 18.9 mm
- net LED_C6: track 273.6 -> 315.8 mm, vias 10 -> 13
- net LED_R9: track 97.9 -> 139.4 mm
- net Net-(J10-Pin_4): track 3.36 -> 37.8 mm
- net LED_R1: track 136.9 -> 105.0 mm, vias 10 -> 3
- net LED_R6: track 95.0 -> 126.1 mm, vias 3 -> 2
- net LED_C5: track 283.6 -> 314.5 mm, vias 10 -> 13
- net Net-(J10-Pin_3): track 3.36 -> 33.1 mm
- net LED_C1: track 308.1 -> 337.0 mm
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Other:
- board size 111.1 x 92.7 mm -> 99.7 x 100.3 mm
- board text added: "1 2 3 4 LED"
- board text added: "A F B G E C D DP"
- board text added: "BU5004"
- board text added: "CA A F B G C E DP D CA"
- board text added: "GL9A040G"
- board text added: "HT16K33"
- board text added: "PCA9306"
- board text added: "SPI for LCD"
- board text removed: "LED 1 2 3 4"
- board text removed: "Molex-105017-0001"
