File: jhl_synth0.kicad_sch (KiCad schematic)
At the start: 5 parts, among them SW1 SW_SPST, U1 YAAJ_BluePill, U2 YAAJ_BlackPill

Commit message: 作図中
Parts:
- removed SW1: SW_SPST, Button_Switch_SMD:SW_Push_1P1T_XKB_TS-1187A, symbol Switch:SW_SPST
- added J1, J3, J4: Conn_01x04, Connector_PinSocket_2.54mm:PinSocket_1x04_P2.54mm_Vertical, symbol Connector_Generic:Conn_01x04
- added J7: Conn_01x07, Connector_PinSocket_2.54mm:PinSocket_1x07_P2.54mm_Vertical, symbol Connector_Generic:Conn_01x07
- added JP1, JP2: SolderJumper_2_Bridged, Jumper:SolderJumper-2_P1.3mm_Bridged_RoundedPad1.0x1.5mm, symbol Jumper:SolderJumper_2_Bridged
- added U3: NUCLEO-F303K8, NUCLEO-F303K8:MODULE_NUCLEO-F303K8, symbol NUCLEO-F303K8:NUCLEO-F303K8
Connections:
- net +3.3V: now also J1.3 (Pin_3), J3.2 (Pin_2), J4.2 (Pin_2), J7.2 (Pin_2), JP1.1 (A), U3.4_14 (+3V3)
- net +5VP: now also U3.4_4 (+5V)
- net GND: now also J1.4 (Pin_4), J3.1 (Pin_1), J4.1 (Pin_1), J7.1 (Pin_1), U3.3_4 (GND_1), U3.4_2 (GND_2)
- net a0: now also U3.4_12 (PA0)
- net a1: now also U3.4_11 (PA1)
- net a2: now also U3.4_10 (PA3)
- net a3: now also JP2.1 (A), U3.4_9 (PA4)
- net a4: now also U3.4_8 (PA5)
- net sw3: now reaches A2.10 (D7)
- net sw3: now also A1.22 (D7)
- net sw4: now reaches A2.11 (D8)
- net sw4: now also A1.23 (D8)
- net sw5: now reaches A2.12 (D9)
- net sw5: now also A1.24 (D9)
- net avref: now reaches A2.18 (AREF)
- net avref: now also A1.30 (AREF), JP1.2 (B)
- net I2C_SDA: now reaches A2.5 (D2)
- net I2C_SDA: now also A1.17 (D2/SDA), U1.15 (PB7), U2.15 (PB7), J1.2 (Pin_2), J3.4 (Pin_4), J4.4 (Pin_4)
- net I2C_SCL: now reaches A2.6 (D3)
- net I2C_SCL: now also A1.18 (D3/SCL), U1.14 (PB6), U2.14 (PB6), J1.1 (Pin_1), J3.3 (Pin_3), J4.3 (Pin_3)
- net sw0: now reaches A2.7 (D4)
- net sw0: now also A1.19 (D4)
- net sw1: now reaches A2.8 (D5)
- net sw1: now also A1.20 (D5)
- net sw2: now reaches A2.9 (D6)
- net sw2: now also A1.21 (D6)
- net SPI_SS: now reaches U2.10 (PA15)
- net SPI_SS: now also U1.10 (PA15), J7.7 (Pin_7), JP2.2 (B)
- net a5 renamed SPI_SCLK
- net SPI_SCLK: now also J7.3 (Pin_3), U3.4_15 (PB3), U3.4_7 (PA6)
- net a6 renamed SPI_MOSI
- net SPI_MOSI: now also J7.4 (Pin_4), U3.3_14 (PB5), U3.4_6 (PA7)
- net a7 renamed SPI_MISO
- net SPI_MISO: now also J7.6 (Pin_6), U3.3_15 (PB4), U3.4_5 (PA2)
- new net spi_lcd_res: J7.5 (Pin_5)
Other:
- sheet pots ports: added sw0, sw1, sw2, sw3, sw4, sw5; removed none
- moved on the sheet: U2

Commit message: 仮回路、仮配置
Parts:
- added J2: USB_B_Micro, Connector_USB:USB_Micro-B_Molex-105017-0001, symbol Connector:USB_B_Micro
- added J5: Conn_01x01, Connector_PinSocket_2.54mm:PinSocket_1x01_P2.54mm_Vertical, symbol Connector_Generic:Conn_01x01
- added JP3, JP4: SolderJumper_2_Bridged, Jumper:SolderJumper-2_P1.3mm_Bridged_RoundedPad1.0x1.5mm, symbol Jumper:SolderJumper_2_Bridged
Connections:
- net +5VP: now also J2.1 (VBUS)
- net GND: now also J2.5 (GND)
- net I2C_SCL: now also U3.3_8 (PB6)
- net I2C_SDA: now also U3.3_7 (PB7)
- net SPI_MISO: now also U1.12 (PB4), U2.12 (PB4); no longer A2.26 (A7), U1.32 (PA7), U2.30 (PA7), U3.4_5 (PA2)
- net SPI_MOSI: now also U1.13 (PB5), U2.13 (PB5); no longer A2.25 (A6), U1.31 (PA6), U2.29 (PA6), U3.4_6 (PA7)
- net SPI_SCLK: now also U1.11 (PB3), U2.11 (PB3); no longer A1.14 (A5), A2.24 (A5), U1.30 (PA5), U2.28 (PA5), U3.4_7 (PA6)
- net sw3: now also U1.2 (PB13), U2.2 (PB13)
- net sw4: now also U1.3 (PB14), U2.3 (PB14)
- net sw5: now also U1.4 (PB15), U2.4 (PB15)
- net USB_DM: now reaches U2.8 (PA11)
- net USB_DM: now also U1.8 (PA11), JP4.1 (A)
- net USB_DP: now reaches U2.9 (PA12)
- net USB_DP: now also U1.9 (PA12), JP3.1 (A)
- new net: J2.2 (D-), JP4.2 (B)
- new net: J2.3 (D+), JP3.2 (B)
- new net: J2.4 (ID), J5.1 (Pin_1)
- new net a5: A1.14 (A5), A2.24 (A5), U1.30 (PA5), U2.28 (PA5), U3.4_7 (PA6)
- new net a6: A2.25 (A6), U1.31 (PA6), U2.29 (PA6), U3.4_6 (PA7)
- new net a7: A2.26 (A7), U1.32 (PA7), U2.30 (PA7), U3.4_5 (PA2)
Other:
- moved on the sheet: U1, U2

Commit message: 日々の進捗
Parts:
- removed J7: Conn_01x07, Connector_PinSocket_2.54mm:PinSocket_1x07_P2.54mm_Vertical, symbol Connector_Generic:Conn_01x07
- added J7: Conn_01x08, Connector_PinHeader_2.54mm:PinHeader_1x08_P2.54mm_Vertical, symbol Connector_Generic:Conn_01x08
- added JP5, JP6: SolderJumper_3_Bridged12, Jumper:SolderJumper-3_P1.3mm_Bridged12_RoundedPad1.0x1.5mm, symbol Jumper:SolderJumper_3_Bridged12
Connections:
- net +3.3V: now also J7.2 (Pin_2), JP5.3 (B), JP6.1 (A); no longer J3.2 (Pin_2)
- net GND: now also J7.1 (Pin_1), JP5.1 (A), JP6.3 (B); no longer J3.1 (Pin_1)
- net SPI_MISO: now also J7.6 (Pin_6)
- net SPI_MOSI: now also J7.4 (Pin_4)
- net SPI_SCLK: now also J7.3 (Pin_3)
- net SPI_SS: now also J7.7 (Pin_7)
- net spi_lcd_res: now also J7.5 (Pin_5)
- new net: J3.2 (Pin_2), JP5.2 (C)
- new net: J3.1 (Pin_1), JP6.2 (C)
- new net LCD_BLK: J7.8 (Pin_8)
Other:
- added sheet leds (leds.kicad_sch)
- moved on the sheet: J4

Commit message: 251023
Parts:
- removed J3, J4: Conn_01x04, Connector_PinSocket_2.54mm:PinSocket_1x04_P2.54mm_Vertical, symbol Connector_Generic:Conn_01x04
- removed JP1, JP2, JP3, JP4: SolderJumper_2_Bridged, Jumper:SolderJumper-2_P1.3mm_Bridged_RoundedPad1.0x1.5mm, symbol Jumper:SolderJumper_2_Bridged
- removed JP5, JP6: SolderJumper_3_Bridged12, Jumper:SolderJumper-3_P1.3mm_Bridged12_RoundedPad1.0x1.5mm, symbol Jumper:SolderJumper_3_Bridged12
- removed U3: NUCLEO-F303K8, NUCLEO-F303K8:MODULE_NUCLEO-F303K8, symbol NUCLEO-F303K8:NUCLEO-F303K8
- added A1: Arduino_Leonardo, Module:Arduino_UNO_R3, symbol MCU_Module:Arduino_Leonardo
- added J1, J11, J12, J13, J14, J15, J16, J17, J19, J21, J22, J23, J24, J25, J26, J28, J29, J3: Conn_01x01, Connector_PinSocket_2.54mm:PinSocket_1x01_P2.54mm_Vertical, symbol Connector_Generic:Conn_01x01
- added J10, J18, J27, J7, J9: Conn_01x04, Connector_PinSocket_2.54mm:PinSocket_1x04_P2.54mm_Vertical, symbol Connector_Generic:Conn_01x04
- added J20, J30: Conn_02x05_Odd_Even, Connector_PinHeader_2.54mm:PinHeader_2x05_P2.54mm_Vertical, symbol Connector_Generic:Conn_02x05_Odd_Even
- added J6: Conn_01x08, Connector_PinHeader_2.54mm:PinHeader_1x08_P2.54mm_Vertical, symbol Connector_Generic:Conn_01x08
- renumbered A1 to A2, A2 to A3, J5 to J4, J7 to J5, J1 to J8, U2 to U1, U1 to U2
Connections:
- net +3.3V: now also J20.1 (Pin_1), J20.10 (Pin_10), J20.2 (Pin_2), J20.3 (Pin_3), J20.4 (Pin_4), J20.5 (Pin_5), J20.6 (Pin_6), J20.7 (Pin_7), J20.8 (Pin_8), J20.9 (Pin_9); no longer A2.4 (3V3), J5.2 (Pin_2), J8.3 (Pin_3), U2.20 (3V3), U2.38 (3V3)
- net +5VP: no longer A2.5 (+5V), U2.18 (5V)
- net GND: now also J30.1 (Pin_1), J30.10 (Pin_10), J30.2 (Pin_2), J30.3 (Pin_3), J30.4 (Pin_4), J30.5 (Pin_5), J30.6 (Pin_6), J30.7 (Pin_7), J30.8 (Pin_8), J30.9 (Pin_9); no longer A2.29 (GND), A2.6 (GND), A2.7 (GND), A3.29 (GND), A3.4 (GND), J5.1 (Pin_1), J8.4 (Pin_4), U1.17 (GND), U1.18 (GND), U2.19 (GND), U2.39 (GND), U2.40 (GND)
- net I2C_SCL: now also J27.1 (Pin_1), J27.2 (Pin_2), J27.3 (Pin_3), J27.4 (Pin_4); no longer A2.18 (D3/SCL), A3.6 (D3), J8.1 (Pin_1), U1.14 (PB6), U2.14 (PB6)
- net I2C_SDA: now also J18.1 (Pin_1), J18.2 (Pin_2), J18.3 (Pin_3), J18.4 (Pin_4); no longer A2.17 (D2/SDA), A3.5 (D2), J8.2 (Pin_2), U1.15 (PB7), U2.15 (PB7)
- net at J2.2 (D-): now also J3.1 (Pin_1)
- net at J2.3 (D+): now also J1.1 (Pin_1)
- net at A2.15 (D0/RX): now also A1.15 (D0/RX)
- net at A2.16 (D1/TX): now also A1.16 (D1/TX)
- net at A2.2 (IOREF): now also A1.2 (IOREF)
- net at A2.25 (D10): now also A1.25 (D10)
- net at A2.26 (D11): now also A1.26 (D11)
- net at A2.27 (D12): now also A1.27 (D12)
- net at A2.28 (D13): now also A1.28 (D13)
- net at A2.3 (~{RESET}): now also A1.3 (~{RESET})
- net at A2.31 (SDA/D2): now also A1.31 (SDA/D2)
- net at A2.32 (SCL/D3): now also A1.32 (SCL/D3)
- net at A2.8 (VIN): now also A1.8 (VIN)
- net LCD_BLK: no longer names the net of J5.8 (Pin_8)
- net LCD_BLK: now also J6.8 (Pin_8)
- removed net SPI_MISO: J5.6 (Pin_6), U1.12 (PB4), U2.12 (PB4)
- removed net SPI_MOSI: J5.4 (Pin_4), U1.13 (PB5), U2.13 (PB5)
- removed net SPI_SCLK: J5.3 (Pin_3), U1.11 (PB3), U2.11 (PB3)
- removed net SPI_SS: J5.7 (Pin_7), U1.10 (PA15), U2.10 (PA15)
- net USB_DM: no longer names the net of U1.8 (PA11)
- net USB_DM: no longer U2.8 (PA11)
- net USB_DP: no longer names the net of U1.9 (PA12)
- net USB_DP: no longer U2.9 (PA12)
- removed net a0: A2.9 (A0), A3.19 (A0), U1.23 (PA0), U2.25 (PA0)
- removed net a1: A2.10 (A1), A3.20 (A1), U1.24 (PA1), U2.26 (PA1)
- removed net a2: A2.11 (A2), A3.21 (A2), U1.25 (PA2), U2.27 (PA2)
- removed net a3: A2.12 (A3), A3.22 (A3), U1.26 (PA3), U2.28 (PA3)
- removed net a4: A2.13 (A4), A3.23 (A4), U1.27 (PA4), U2.29 (PA4)
- removed net a5: A2.14 (A5), A3.24 (A5), U1.28 (PA5), U2.30 (PA5)
- removed net a6: A3.25 (A6), U1.29 (PA6), U2.31 (PA6)
- removed net a7: A3.26 (A7), U1.30 (PA7), U2.32 (PA7)
- net a8: no longer names the net of U1.31 (PB0)
- net a8: no longer U2.33 (PB0)
- net a9: no longer names the net of U1.32 (PB1)
- net a9: no longer U2.34 (PB1)
- net avref: no longer names the net of A3.18 (AREF)
- net avref: no longer A2.30 (AREF)
- net spi_lcd_res: no longer names the net of J5.5 (Pin_5)
- net spi_lcd_res: now also J6.5 (Pin_5)
- net sw0: no longer names the net of A3.7 (D4)
- net sw0: no longer A2.19 (D4)
- net sw1: no longer names the net of A3.8 (D5)
- net sw1: no longer A2.20 (D5)
- net sw2: no longer names the net of A3.9 (D6)
- net sw2: no longer A2.21 (D6)
- removed net sw3: A2.22 (D7), A3.10 (D7), U1.2 (PB13), U2.2 (PB13)
- removed net sw4: A2.23 (D8), A3.11 (D8), U1.3 (PB14), U2.3 (PB14)
- removed net sw5: A2.24 (D9), A3.12 (D9), U1.4 (PB15), U2.4 (PB15)
- new net: J7.1 (Pin_1), J8.1 (Pin_1)
- new net: J7.2 (Pin_2), J8.2 (Pin_2)
- new net: J7.3 (Pin_3), J8.3 (Pin_3)
- new net: J7.4 (Pin_4), J8.4 (Pin_4)
- new net: J5.1 (Pin_1), J6.1 (Pin_1)
- new net: J5.2 (Pin_2), J6.2 (Pin_2)
- new net: J5.3 (Pin_3), J6.3 (Pin_3)
- new net: J5.4 (Pin_4), J6.4 (Pin_4)
- new net: J5.6 (Pin_6), J6.6 (Pin_6)
- new net: J5.7 (Pin_7), J6.7 (Pin_7)
- new net: J10.1 (Pin_1), J9.1 (Pin_1)
- new net: J10.2 (Pin_2), J9.2 (Pin_2)
- new net: J10.3 (Pin_3), J9.3 (Pin_3)
- new net: J10.4 (Pin_4), J9.4 (Pin_4)
- new net: A1.10 (A1), A2.10 (A1)
- new net: A1.11 (A2), A2.11 (A2)
- new net: A1.12 (A3), A2.12 (A3)
- new net: A1.13 (A4), A2.13 (A4)
- new net: A1.14 (A5), A2.14 (A5)
- new net: A1.17 (D2/SDA), A2.17 (D2/SDA)
- new net: A1.18 (D3/SCL), A2.18 (D3/SCL)
- new net: A1.19 (D4), A2.19 (D4)
- new net: A1.20 (D5), A2.20 (D5)
- new net: A1.21 (D6), A2.21 (D6)
- new net: A1.22 (D7), A2.22 (D7)
- new net: A1.23 (D8), A2.23 (D8)
- new net: A1.24 (D9), A2.24 (D9)
- new net: A1.29 (GND), A2.29 (GND)
- new net: A1.30 (AREF), A2.30 (AREF)
- new net: A1.4 (3V3), A2.4 (3V3)
- new net: A1.5 (+5V), A2.5 (+5V)
- new net: A1.6 (GND), A2.6 (GND)
- new net: A1.7 (GND), A2.7 (GND)
- new net: A1.9 (A0), A2.9 (A0)
- new net pots/a0: J11.1 (Pin_1)
- new net pots/a1: J12.1 (Pin_1)
- new net pots/a2: J13.1 (Pin_1)
- new net pots/a3: J14.1 (Pin_1)
- new net pots/a4: J15.1 (Pin_1)
- new net pots/a5: J16.1 (Pin_1)
- new net pots/a6: J17.1 (Pin_1)
- new net pots/a7: J19.1 (Pin_1)
- new net pots/a8: J21.1 (Pin_1)
- new net pots/a9: J22.1 (Pin_1)
- new net pots/sw0: J23.1 (Pin_1)
- new net pots/sw1: J24.1 (Pin_1)
- new net pots/sw2: J25.1 (Pin_1)
- new net pots/sw3: J26.1 (Pin_1)
- new net pots/sw4: J28.1 (Pin_1)
- new net pots/sw5: J29.1 (Pin_1)
Other:
- added sheet conns (conns.kicad_sch)
- moved on the sheet: J4

Commit message: 更新
Parts:
- added D100, D97, D98, D99: LED_Small_Filled, LED_SMD:LED_0603_1608Metric_Pad1.05x0.95mm_HandSolder, symbol Device:LED_Small_Filled
- added J35: Conn_01x04, Connector_PinSocket_2.54mm:PinSocket_1x04_P2.54mm_Vertical, symbol Connector_Generic:Conn_01x04
- added R1, R2, R3, R4: R_Small_US, Resistor_SMD:R_0402_1005Metric_Pad0.72x0.64mm_HandSolder, symbol Device:R_Small_US
Connections:
- net GND: now also D100.1 (K), D97.1 (K), D98.1 (K), D99.1 (K)
- new net: J35.1 (Pin_1), R1.1
- new net: D97.2 (A), R1.2
- new net: J35.2 (Pin_2), R2.1
- new net: J35.3 (Pin_3), R3.1
- new net: J35.4 (Pin_4), R4.1
- new net: D98.2 (A), R2.2
- new net: D99.2 (A), R3.2
- new net: D100.2 (A), R4.2

Commit message: 更新
Parts:
- J10, J11, J12, J13, J14, J15, J16, J17, J18, J19, J20, J21, J22, J23, J24, J25, J26, J27, J28, J29, J30, J35, J5, J6, J7, J8, J9: now not fitted
Changed lines of the file:
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@@
 		(in_bom yes)
 		(on_board yes)
-		(dnp no)
+		(dnp yes)
 		(fields_autoplaced yes)
 		(property "Reference" "J20"
@@
 		(in_bom yes)
 		(on_board yes)
-		(dnp no)
+		(dnp yes)
 		(property "Reference" "J29"
 			(at 251.714 150.876 0)
@@
 		(in_bom yes)
 		(on_board yes)
-		(dnp no)
+		(dnp yes)
 		(property "Reference" "J14"
 			(at 251.714 117.856 0)
@@
 		(in_bom yes)
 		(on_board yes)
-		(dnp no)
+		(dnp yes)
 		(property "Reference" "J35"
 			(at 218.186 76.454 0)
@@
 		(in_bom yes)
 		(on_board yes)
-		(dnp no)
+		(dnp yes)
 		(property "Reference" "J27"
 			(at 192.024 139.446 0)
@@
 		(in_bom yes)
 		(on_board yes)
-		(dnp no)
+		(dnp yes)
 		(property "Reference" "J25"
 			(at 251.714 143.256 0)
@@
 		(in_bom yes)
 		(on_board yes)
-		(dnp no)
+		(dnp yes)
 		(property "Reference" "J7"
 			(at 251.206 76.454 0)
@@
 		(in_bom yes)
 		(on_board yes)
-		(dnp no)
+		(dnp yes)
 		(property "Reference" "J19"
 			(at 251.714 128.016 0)
@@
 		(in_bom yes)
 		(on_board yes)
-		(dnp no)
+		(dnp yes)
 		(fields_autoplaced yes)
 		(property "Reference" "J6"
@@
 		(in_bom yes)
 		(on_board yes)
-		(dnp no)
+		(dnp yes)
 		(property "Reference" "J11"
 			(at 251.714 110.236 0)
@@
 		(in_bom yes)
 		(on_board yes)
-		(dnp no)
+		(dnp yes)
 		(property "Reference" "J15"
 			(at 251.714 120.396 0)
@@
 		(in_bom yes)
 		(on_board yes)
-		(dnp no)
+		(dnp yes)
 		(property "Reference" "J22"
 			(at 251.714 133.096 0)
@@
 		(in_bom yes)
 		(on_board yes)
-		(dnp no)
+		(dnp yes)
 		(property "Reference" "J18"
 			(at 192.024 120.396 0)
@@
 		(in_bom yes)
 		(on_board yes)
-		(dnp no)
+		(dnp yes)
 		(property "Reference" "J26"
 			(at 251.714 145.796 0)
@@
 		(in_bom yes)
 		(on_board yes)
-		(dnp no)
+		(dnp yes)
 		(property "Reference" "J21"
 			(at 251.714 130.556 0)
@@
 		(in_bom yes)
 		(on_board yes)
-		(dnp no)
+		(dnp yes)
 		(property "Reference" "J9"
 			(at 215.646 92.456 0)
@@
 		(in_bom yes)
 		(on_board yes)
-		(dnp no)
+		(dnp yes)
 		(property "Reference" "J23"
 			(at 251.714 138.176 0)
@@
 		(in_bom yes)
 		(on_board yes)
-		(dnp no)
+		(dnp yes)
 		(property "Reference" "J5"
 			(at 255.27 43.1799 0)
@@
 		(in_bom yes)
 		(on_board yes)
-		(dnp no)
+		(dnp yes)
 		(property "Reference" "J12"
 			(at 251.714 112.776 0)
@@
 		(in_bom yes)
 		(on_board yes)
-		(dnp no)
+		(dnp yes)
 		(property "Reference" "J28"
 			(at 251.714 148.336 0)
@@
 		(in_bom yes)
 		(on_board yes)
-		(dnp no)
+		(dnp yes)
 		(fields_autoplaced yes)
 		(property "Reference" "J30"
@@
 		(in_bom yes)
 		(on_board yes)
-		(dnp no)
+		(dnp yes)
 		(property "Reference" "J24"
 			(at 251.714 140.716 0)
@@
 		(in_bom yes)
 		(on_board yes)
-		(dnp no)
+		(dnp yes)
 		(property "Reference" "J16"
 			(at 251.714 122.936 0)
@@
 		(in_bom yes)
 		(on_board yes)
-		(dnp no)
+		(dnp yes)
 		(property "Reference" "J8"
 			(at 260.604 76.454 0)
@@
 		(in_bom yes)
 		(on_board yes)
-		(dnp no)
+		(dnp yes)
 		(property "Reference" "J17"
 			(at 251.714 125.476 0)
@@
 		(in_bom yes)
 		(on_board yes)
-		(dnp no)
+		(dnp yes)
 		(property "Reference" "J10"
 			(at 225.044 92.456 0)
@@
 		(in_bom yes)
 		(on_board yes)
-		(dnp no)
+		(dnp yes)
 		(property "Reference" "J13"
 			(at 251.714 115.316 0)
