File: jhl_synth0.kicad_sch (KiCad schematic)
At the start: 44 parts, among them J1 Conn_01x01, J10 Conn_01x04, J11 Conn_01x01, J12 Conn_01x01, J13 Conn_01x01, J14 Conn_01x01, J15 Conn_01x01, J16 Conn_01x01, J17 Conn_01x01, J18 Conn_01x04, J19 Conn_01x01, J2 USB_B_Micro, J20 Conn_02x05_Odd_Even, J21 Conn_01x01, J22 Conn_01x01, J23 Conn_01x01, J24 Conn_01x01, J25 Conn_01x01, J26 Conn_01x01, J27 Conn_01x04, J28 Conn_01x01, J29 Conn_01x01, J3 Conn_01x01, J30 Conn_02x05_Odd_Even, J35 Conn_01x04, J4 Conn_01x01, J5 Conn_01x08, J6 Conn_01x08, J7 Conn_01x04, J8 Conn_01x04, J9 Conn_01x04, U1 YAAJ_BlackPill, U2 YAAJ_BluePill

Commit message: 更新
Parts:
- added H1, H2, H3, H4: MountingHole, MountingHole:MountingHole_3.2mm_M3, symbol Mechanical:MountingHole
- added J45, J46, J47, J48: Conn_01x01, Connector_PinSocket_2.54mm:PinSocket_1x01_P2.54mm_Vertical, symbol Connector_Generic:Conn_01x01
Connections:
- new net pots/sw6: J45.1 (Pin_1)
- new net pots/sw7: J46.1 (Pin_1)
- new net pots/sw8: J47.1 (Pin_1)
- new net pots/sw9: J48.1 (Pin_1)
Other:
- sheet pots ports: added sw6, sw7, sw8, sw9; removed none

Commit message: 更新
Parts:
- added J51: Conn_01x08, Connector_PinHeader_2.54mm:PinHeader_1x08_P2.54mm_Vertical, symbol Connector_Generic:Conn_01x08
- added J52: Conn_01x04, Connector_PinSocket_2.54mm:PinSocket_1x04_P2.54mm_Vertical, symbol Connector_Generic:Conn_01x04
- J2: footprint Connector_USB:USB_Micro-B_Molex-105017-0001 -> libs:usb b micro jhl
Connections:
- net at J10.1 (Pin_1), J9.1 (Pin_1): now also J52.1 (Pin_1)
- net at J10.2 (Pin_2), J9.2 (Pin_2): now also J52.2 (Pin_2)
- net at J10.3 (Pin_3), J9.3 (Pin_3): now also J52.3 (Pin_3)
- net at J10.4 (Pin_4), J9.4 (Pin_4): now also J52.4 (Pin_4)
- new net LED_C0_d: J51.1 (Pin_1)
- new net LED_C1_d: J51.2 (Pin_2)
- new net LED_C2_d: J51.3 (Pin_3)
- new net LED_C3_d: J51.4 (Pin_4)
- new net LED_C4_d: J51.5 (Pin_5)
- new net LED_C5_d: J51.6 (Pin_6)
- new net LED_C6_d: J51.7 (Pin_7)
- new net LED_C7_d: J51.8 (Pin_8)
Other:
- moved on the sheet: A1, A3
