File: leds.kicad_sch (KiCad schematic)
At the start: 6 parts, among them IC1 HT16K33

Commit message: 251023
Parts:
- added D11, D12, D13, D14, D15, D16, D17, D18, D19, D20, D21, D22, D23, D24, D25, D26, D27, D28, D29, D3, D30, D31, D32, D33, D34, D35, D36, D37, D38, D39, D4, D40, D41, D42, D43, D44, D45, D46, D47, D48, D49, D5, D50, D51, D52, D53, D54, D55, D56, D57, D58, D59, D6, D60, D61, D62, D63, D64, D65, D66, D67, D68, D69, D7, D70, D71, D72, D73, D74, D75, D76, D77, D78, D79, D8, D80, D81, D82, D83, D84, D85, D86, D87, D88, D89, D90, D91, D92, D93, D94, D95, D96: LED_Small_Filled, LED_SMD:LED_0603_1608Metric_Pad1.05x0.95mm_HandSolder, symbol Device:LED_Small_Filled
- renumbered D4 to D10, D3 to D9
Connections:
- net at D10.1 (K), D2.1 (K), IC1.3 (COM1/KS0): now also D18.1 (K), D26.1 (K), D34.1 (K), D42.1 (K), D50.1 (K), D58.1 (K), D66.1 (K), D74.1 (K), D82.1 (K), D90.1 (K)
- net at D10.2 (A), D9.2 (A), IC1.20 (ROW1/A0): now also D11.2 (A), D12.2 (A), D13.2 (A), D14.2 (A), D15.2 (A), D16.2 (A)
- net at D1.2 (A), D2.2 (A), IC1.21 (ROW0/A1): now also D3.2 (A), D4.2 (A), D5.2 (A), D6.2 (A), D7.2 (A), D8.2 (A)
- net at IC1.10 (ROW11/K10/INT): now also D89.2 (A), D90.2 (A), D91.2 (A), D92.2 (A), D93.2 (A), D94.2 (A), D95.2 (A), D96.2 (A)
- net at IC1.11 (ROW10/K9): now also IC1.4 (COM2/KS1), D11.1 (K), D19.1 (K), D27.1 (K), D3.1 (K), D35.1 (K), D43.1 (K), D51.1 (K), D59.1 (K), D67.1 (K), D75.1 (K), D81.2 (A), D82.2 (A), D83.1 (K), D83.2 (A), D84.2 (A), D85.2 (A), D86.2 (A), D87.2 (A), D88.2 (A), D91.1 (K)
- net at IC1.12 (ROW9/K8): now also D73.2 (A), D74.2 (A), D75.2 (A), D76.2 (A), D77.2 (A), D78.2 (A), D79.2 (A), D80.2 (A)
- net at IC1.13 (ROW8/K7): now also D65.2 (A), D66.2 (A), D67.2 (A), D68.2 (A), D69.2 (A), D70.2 (A), D71.2 (A), D72.2 (A)
- net at IC1.14 (ROW7/K6): now also D57.2 (A), D58.2 (A), D59.2 (A), D60.2 (A), D61.2 (A), D62.2 (A), D63.2 (A), D64.2 (A)
- net at IC1.15 (ROW6/K5): now also D49.2 (A), D50.2 (A), D51.2 (A), D52.2 (A), D53.2 (A), D54.2 (A), D55.2 (A), D56.2 (A)
- net at IC1.16 (ROW5/K4): now also D41.2 (A), D42.2 (A), D43.2 (A), D44.2 (A), D45.2 (A), D46.2 (A), D47.2 (A), D48.2 (A)
- net at IC1.17 (ROW4/K3): now also D33.2 (A), D34.2 (A), D35.2 (A), D36.2 (A), D37.2 (A), D38.2 (A), D39.2 (A), D40.2 (A)
- net at IC1.18 (ROW3/K2): now also D25.2 (A), D26.2 (A), D27.2 (A), D28.2 (A), D29.2 (A), D30.2 (A), D31.2 (A), D32.2 (A)
- net at IC1.19 (ROW2/K1): now also D17.2 (A), D18.2 (A), D19.2 (A), D20.2 (A), D21.2 (A), D22.2 (A), D23.2 (A), D24.2 (A)
- net at D1.1 (K), D9.1 (K), IC1.2 (COM0/AD): now also D17.1 (K), D25.1 (K), D33.1 (K), D41.1 (K), D49.1 (K), D57.1 (K), D65.1 (K), D73.1 (K), D81.1 (K), D89.1 (K)
- net at IC1.5 (COM3/KS2): now also D12.1 (K), D20.1 (K), D28.1 (K), D36.1 (K), D4.1 (K), D44.1 (K), D52.1 (K), D60.1 (K), D68.1 (K), D76.1 (K), D84.1 (K), D92.1 (K)
- net at IC1.6 (COM4): now also D13.1 (K), D21.1 (K), D29.1 (K), D37.1 (K), D45.1 (K), D5.1 (K), D53.1 (K), D61.1 (K), D69.1 (K), D77.1 (K), D85.1 (K), D93.1 (K)
- net at IC1.7 (COM5): now also D14.1 (K), D22.1 (K), D30.1 (K), D38.1 (K), D46.1 (K), D54.1 (K), D6.1 (K), D62.1 (K), D70.1 (K), D78.1 (K), D86.1 (K), D94.1 (K)
- net at IC1.8 (COM6): now also D15.1 (K), D23.1 (K), D31.1 (K), D39.1 (K), D47.1 (K), D55.1 (K), D63.1 (K), D7.1 (K), D71.1 (K), D79.1 (K), D87.1 (K), D95.1 (K)
- net at IC1.9 (COM7): now also D16.1 (K), D24.1 (K), D32.1 (K), D40.1 (K), D48.1 (K), D56.1 (K), D64.1 (K), D72.1 (K), D8.1 (K), D80.1 (K), D88.1 (K), D96.1 (K)
Other:
- moved on the sheet: C1, D1, D10, D2, D9, IC1

Commit message: 更新
Parts:
- added D101: ~, libs:BU5004, symbol JHLLibrary:led_matrix_8x8
- added R5: R_Small_US, Resistor_SMD:R_0402_1005Metric_Pad0.72x0.64mm_HandSolder, symbol Device:R_Small_US
- added U3, U4, U7: SA39-12SRWA, Display_7Segment:Sx39-1xxxxx, symbol Display_Character:SA39-12SRWA
- added U5: PCA9306DC, Package_SO:VSSOP-8_2.3x2mm_P0.5mm, symbol Interface:PCA9306DC
- added U6: PCA9306DP, Package_SO:TSSOP-8_3x3mm_P0.65mm, symbol Interface:PCA9306DP
Connections:
- net +3.3V: now also U5.2 (VREF1), U6.2 (VREF1); no longer C1.1, IC1.24 (VDD)
- net GND: now also U5.1 (GND), U6.1 (GND)
- net I2C_SCL: now also U5.3 (SCL1), U6.3 (SCL1)
- net I2C_SDA: now also U5.4 (SDA1), U6.4 (SDA1)
- net LED_C5: now reaches D14.1 (K), D22.1 (K), D30.1 (K), D38.1 (K), D46.1 (K), D54.1 (K), D6.1 (K), D62.1 (K), D70.1 (K), D78.1 (K), D86.1 (K), D94.1 (K), IC1.7 (COM5)
- net LED_C5: now also D101.11 (COL6), U3.2 (F), U4.2 (F), U7.2 (F)
- net LED_R7: now reaches D57.2 (A), D58.2 (A), D59.2 (A), D60.2 (A), D61.2 (A), D62.2 (A), D63.2 (A), D64.2 (A), IC1.14 (ROW7/K6)
- net LED_R7: now also D101.8 (ROW8)
- net LED_C7: now reaches D16.1 (K), D24.1 (K), D32.1 (K), D40.1 (K), D48.1 (K), D56.1 (K), D64.1 (K), D72.1 (K), D8.1 (K), D80.1 (K), D88.1 (K), D96.1 (K), IC1.9 (COM7)
- net LED_C7: now also D101.15 (COL8), U3.7 (DP), U4.7 (DP), U7.7 (DP)
- net LED_R6: now reaches D49.2 (A), D50.2 (A), D51.2 (A), D52.2 (A), D53.2 (A), D54.2 (A), D55.2 (A), D56.2 (A), IC1.15 (ROW6/K5)
- net LED_R6: now also D101.9 (ROW7)
- net LED_C6: now reaches D15.1 (K), D23.1 (K), D31.1 (K), D39.1 (K), D47.1 (K), D55.1 (K), D63.1 (K), D7.1 (K), D71.1 (K), D79.1 (K), D87.1 (K), D95.1 (K), IC1.8 (COM6)
- net LED_C6: now also D101.12 (COL7), U3.3 (G), U4.3 (G), U7.3 (G)
- net LED_R1: now reaches D10.2 (A), D11.2 (A), D12.2 (A), D13.2 (A), D14.2 (A), D15.2 (A), D16.2 (A), D9.2 (A), IC1.20 (ROW1/A0)
- net LED_R1: now also D101.1 (ROW2)
- net LED_C2: now reaches D11.1 (K), D19.1 (K), D27.1 (K), D3.1 (K), D35.1 (K), D43.1 (K), D51.1 (K), D59.1 (K), D67.1 (K), D75.1 (K), D83.1 (K), D91.1 (K), IC1.4 (COM2/KS1)
- net LED_C2: now also D101.3 (COL3), U3.8 (C), U4.8 (C), U7.8 (C); no longer D81.2 (A), D82.2 (A), D83.2 (A), D84.2 (A), D85.2 (A), D86.2 (A), D87.2 (A), D88.2 (A), IC1.11 (ROW10/K9)
- net LED_C4: now reaches D13.1 (K), D21.1 (K), D29.1 (K), D37.1 (K), D45.1 (K), D5.1 (K), D53.1 (K), D61.1 (K), D69.1 (K), D77.1 (K), D85.1 (K), D93.1 (K), IC1.6 (COM4)
- net LED_C4: now also D101.10 (COL5), U3.4 (E), U4.4 (E), U7.4 (E)
- net LED_R9: now reaches D73.2 (A), D74.2 (A), D75.2 (A), D76.2 (A), D77.2 (A), D78.2 (A), D79.2 (A), D80.2 (A), IC1.12 (ROW9/K8)
- net LED_R9: now also U3.1 (CA), U3.6 (CA)
- net LED_R4: now reaches D33.2 (A), D34.2 (A), D35.2 (A), D36.2 (A), D37.2 (A), D38.2 (A), D39.2 (A), D40.2 (A), IC1.17 (ROW4/K3)
- net LED_R4: now also D101.5 (ROW5)
- net LED_R0: now reaches D1.2 (A), D2.2 (A), D3.2 (A), D4.2 (A), D5.2 (A), D6.2 (A), D7.2 (A), D8.2 (A), IC1.21 (ROW0/A1)
- net LED_R0: now also D101.16 (ROW1)
- net LED_C1: now reaches D10.1 (K), D18.1 (K), D2.1 (K), D26.1 (K), D34.1 (K), D42.1 (K), D50.1 (K), D58.1 (K), D66.1 (K), D74.1 (K), D82.1 (K), D90.1 (K), IC1.3 (COM1/KS0)
- net LED_C1: now also D101.4 (COL2), U3.9 (B), U4.9 (B), U7.9 (B)
- net LED_C0: now reaches D1.1 (K), D17.1 (K), D25.1 (K), D33.1 (K), D41.1 (K), D49.1 (K), D57.1 (K), D65.1 (K), D73.1 (K), D81.1 (K), D89.1 (K), D9.1 (K), IC1.2 (COM0/AD)
- net LED_C0: now also D101.7 (COL1), U3.10 (A), U4.10 (A), U7.10 (A)
- net LED_R2: now reaches D17.2 (A), D18.2 (A), D19.2 (A), D20.2 (A), D21.2 (A), D22.2 (A), D23.2 (A), D24.2 (A), IC1.19 (ROW2/K1)
- net LED_R2: now also D101.14 (ROW3)
- net LED_R11: now reaches D89.2 (A), D90.2 (A), D91.2 (A), D92.2 (A), D93.2 (A), D94.2 (A), D95.2 (A), D96.2 (A), IC1.10 (ROW11/K10/INT)
- net LED_R3: now reaches D25.2 (A), D26.2 (A), D27.2 (A), D28.2 (A), D29.2 (A), D30.2 (A), D31.2 (A), D32.2 (A), IC1.18 (ROW3/K2)
- net LED_R3: now also D101.13 (ROW4)
- net LED_R5: now reaches D41.2 (A), D42.2 (A), D43.2 (A), D44.2 (A), D45.2 (A), D46.2 (A), D47.2 (A), D48.2 (A), IC1.16 (ROW5/K4)
- net LED_R5: now also D101.6 (ROW6)
- net LED_C3: now reaches D12.1 (K), D20.1 (K), D28.1 (K), D36.1 (K), D4.1 (K), D44.1 (K), D52.1 (K), D60.1 (K), D68.1 (K), D76.1 (K), D84.1 (K), D92.1 (K), IC1.5 (COM3/KS2)
- net LED_C3: now also D101.2 (COL4), U3.5 (D), U4.5 (D), U7.5 (D)
- net LED_R8: now reaches D65.2 (A), D66.2 (A), D67.2 (A), D68.2 (A), D69.2 (A), D70.2 (A), D71.2 (A), D72.2 (A), IC1.13 (ROW8/K7)
- net LED_R8: now also U4.1 (CA), U4.6 (CA)
- new net: R5.1, U5.8 (EN), U6.8 (EN)
- new net +5VP: C1.1, IC1.24 (VDD), R5.2, U5.7 (VREF2), U6.7 (VREF2)
- new net I2C_SCL5: U5.6 (SCL2), U6.6 (SCL2)
- new net I2C_SDA5: U5.5 (SDA2), U6.5 (SDA2)
- new net LED_R10: D81.2 (A), D82.2 (A), D83.2 (A), D84.2 (A), D85.2 (A), D86.2 (A), D87.2 (A), D88.2 (A), IC1.11 (ROW10/K9), U7.1 (CA), U7.6 (CA)
Other:
- moved on the sheet: C1, D1, D10, D11, D12, D13, D14, D15, D16, D17, D18, D19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

Commit message: 更新
Parts:
- R5: value R_Small_US -> 200k
Changed lines of the file:
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@@
 			)
 		)
-		(property "Value" "R_Small_US"
+		(property "Value" "200k"
 			(at 246.38 68.5799 0)
 			(effects

Commit message: 更新
Parts:
- added J36, J40: Conn_01x04, Connector_PinSocket_2.54mm:PinSocket_1x04_P2.54mm_Vertical, symbol Connector_Generic:Conn_01x04
- D101, U3, U4, U5, U7: now left out of the parts list
Connections:
- net +3.3V: now also J36.1 (Pin_1)
- net +5VP: now also J36.4 (Pin_4), J40.4 (Pin_4)
- net GND: now also J40.1 (Pin_1)
- net I2C_SCL: now also J36.2 (Pin_2)
- net I2C_SCL5: now also J40.3 (Pin_3)
- net I2C_SDA: now also J36.3 (Pin_3)
- net I2C_SDA5: now also J40.2 (Pin_2)
Other:
- note added: "i2c level shift module"

Commit message: 更新
Parts:
- removed J36, J40: Conn_01x04, Connector_PinSocket_2.54mm:PinSocket_1x04_P2.54mm_Vertical, symbol Connector_Generic:Conn_01x04
- added J36, J40, J49: Conn_01x02, Connector_PinHeader_2.54mm:PinHeader_2x01_P2.54mm_Vertical, symbol Connector_Generic:Conn_01x02
- added J53: Conn_02x08_Odd_Even, Connector_PinHeader_2.54mm:PinHeader_2x08_P2.54mm_Vertical, symbol Connector_Generic:Conn_02x08_Odd_Even
- added R10, R11, R12, R13, R6, R7, R8, R9: 200k, Resistor_SMD:R_0402_1005Metric_Pad0.72x0.64mm_HandSolder, symbol Device:R_Small_US
- added U8: PCA9306D, Package_SO:SO-8_3.9x4.9mm_P1.27mm, symbol Interface:PCA9306D
Connections:
- net +3.3V: now also U8.2 (VREF1)
- net +5VP: now also U8.7 (VREF2)
- net GND: now also U8.1 (GND)
- net I2C_SCL: now also U8.3 (SCL1); no longer IC1.22 (SCL)
- net I2C_SCL5: now also IC1.22 (SCL), U8.6 (SCL2)
- net I2C_SDA: now also U8.4 (SDA1); no longer IC1.23 (SDA)
- net I2C_SDA5: now also IC1.23 (SDA), U8.5 (SDA2)
- net LED_C0: now also J53.2 (Pin_2)
- net LED_C1: now also J53.4 (Pin_4)
- net LED_C2: now also J53.6 (Pin_6)
- net LED_C3: now also J53.8 (Pin_8)
- net LED_C4: now also J53.10 (Pin_10)
- net LED_C5: now also J53.12 (Pin_12)
- net LED_C6: now also J53.14 (Pin_14)
- net LED_C7: now also J53.16 (Pin_16)
- net LED_R10: now also J49.1 (Pin_1); no longer U7.1 (CA), U7.6 (CA)
- net LED_R8: now also J36.1 (Pin_1); no longer U4.1 (CA), U4.6 (CA)
- net LED_R9: now also J40.1 (Pin_1); no longer U3.1 (CA), U3.6 (CA)
- net at R5.1, U5.8 (EN), U6.8 (EN): now also U8.8 (EN)
- new net: J49.2 (Pin_2), U7.1 (CA), U7.6 (CA)
- new net: J53.5 (Pin_5), R8.1
- new net: J53.15 (Pin_15), R13.1
- new net: J40.2 (Pin_2), U3.1 (CA), U3.6 (CA)
- new net: J53.9 (Pin_9), R10.1
- new net: J53.13 (Pin_13), R12.1
- new net: J36.2 (Pin_2), U4.1 (CA), U4.6 (CA)
- new net: J53.3 (Pin_3), R7.1
- new net: J53.1 (Pin_1), R6.1
- new net: J53.11 (Pin_11), R11.1
- new net: J53.7 (Pin_7), R9.1
- new net LED_C0_d: R6.2
- new net LED_C1_d: R7.2
- new net LED_C2_d: R8.2
- new net LED_C3_d: R9.2
- new net LED_C4_d: R10.2
- new net LED_C5_d: R11.2
- new net LED_C6_d: R12.2
- new net LED_C7_d: R13.2
Other:
- note removed: "i2c level shift module"
- moved on the sheet: D1, D10, D101, D11, D12, D13, D14, D15, D16, D17, D18, D19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
